Commit message: [rolling] add rotors in urdf

File: robots/rolling/robots/rolling.urdf.xacro (robot description, xacro)
@@ -4,4 +4,8 @@
   <xacro:include filename="$(find rolling)/urdf/rolling_link.urdf.xacro" />
   <xacro:include filename="$(find rolling)/urdf/common.xacro" />
-  <xacro:rolling_base_link child1="1" child2="2" />
+  <xacro:rolling_base_link child1="1" child2="2" child3="3" child4="4" />
+  <xacro:rolling_thrust_link self="1" rotor_direction="1" />
+  <xacro:rolling_thrust_link self="2" rotor_direction="-1"/>
+  <xacro:rolling_thrust_link self="3" rotor_direction="1"/>
+  <xacro:rolling_thrust_link self="4" rotor_direction="-1"/>
 </robot>

File: robots/rolling/urdf/common.xacro (robot description, xacro)
@@ -6,4 +6,6 @@
   <thrust_link name="thrust" />
   <m_f_rate value="-0.0172" /> <!-- drug torque rate -->
+  <xacro:property name="max_force" value="18.0" /> <!-- [N] -->
+  <xacro:property name="min_force" value="1.0" /> <!-- [N] -->
   <!-- friction -->
   <xacro:macro name="friction" params="link">

File: robots/rolling/urdf/rolling_link.urdf.xacro (robot description, xacro)
@@ -3,5 +3,5 @@
     xmlns:xacro="http://www.ros.org/wiki/xacro" name="rolling_link" >
   <xacro:property name="cylinder_radius" value="1.0"/>
-  <xacro:macro name="rolling_base_link" params="child1 child2">
+  <xacro:macro name="rolling_base_link" params="child1 child2 child3 child4">
     <link name="root">
       <inertial>
@@ -32,5 +32,5 @@
         <origin xyz="0 0 0" rpy="${pi / 2} 0 0" />
         <geometry>
-          <cylinder radius="${cylinder_radius}" length="0.3"/>
+          <cylinder radius="${cylinder_radius}" length="0.1"/>
         </geometry>
         <material name="white">
@@ -61,4 +61,144 @@
       <axis xyz="0 0 1"/>
     </joint>
+    ## gimbal
+    <joint name="gimbal${child1}" type="revolute">
+      <limit effort="6.6" lower="-1.57" upper="1.57" velocity="3.0"/>
+      <parent link="base_link"/>
+      <child link="gimbal_link${child1}"/>
+      <origin rpy="0 ${pi/2} 0" xyz="${cylinder_radius} 0 0"/>
+      <axis xyz="1 0 0"/>
+      <dynamics damping="0.8" friction="0.0"/>
+    </joint>
+  <joint name="gimbal${child2}" type="revolute">
+      <limit effort="6.6" lower="-1.57" upper="1.57" velocity="3.0"/>
+      <parent link="base_link"/>
+      <child link="gimbal_link${child2}"/>
+      <origin rpy="0 0 0" xyz="0 0 ${cylinder_radius}"/>
+      <axis xyz="1 0 0"/>
+      <dynamics damping="0.8" friction="0.0"/>
+    </joint>
+    <joint name="gimbal${child3}" type="revolute">
+      <limit effort="6.6" lower="-1.57" upper="1.57" velocity="3.0"/>
+      <parent link="base_link"/>
+      <child link="gimbal_link${child3}"/>
+      <origin rpy="0 ${-pi/2} 0" xyz="${- cylinder_radius} 0 0"/>
+      <axis xyz="1 0 0"/>
+      <dynamics damping="0.8" friction="0.0"/>
+    </joint>
+    <joint name="gimbal${child4}" type="revolute">
+      <limit effort="6.6" lower="-1.57" upper="1.57" velocity="3.0"/>
+      <parent link="base_link"/>
+      <child link="gimbal_link${child4}"/>
+      <origin rpy="0 ${pi} 0" xyz="0 0 ${- cylinder_radius}"/>
+      <axis xyz="1 0 0"/>
+      <dynamics damping="0.8" friction="0.0"/>
+    </joint>
+    #### hardware interface ####
+    <transmission name="joint_tran${child1}">
+      <type>transmission_interface/SimpleTransmission</type>
+      <joint name="gimbal${child1}">
+        <hardwareInterface>hardware_interface/EffortJointInterface</hardwareInterface>
+      </joint>
+      <actuator name="servo${child1}">
+        <hardwareInterface>hardware_interface/EffortJointInterface</hardwareInterface>
+        <mechanicalReduction>1</mechanicalReduction>
+      </actuator>
+    </transmission>
+    <transmission name="joint_tran${child2}">
+      <type>transmission_interface/SimpleTransmission</type>
+      <joint name="gimbal${child2}">
+        <hardwareInterface>hardware_interface/EffortJointInterface</hardwareInterface>
+      </joint>
+      <actuator name="servo${child2}">
+        <hardwareInterface>hardware_interface/EffortJointInterface</hardwareInterface>
+        <mechanicalReduction>1</mechanicalReduction>
+      </actuator>
+    </transmission>
+    <transmission name="joint_tran${child3}">
+      <type>transmission_interface/SimpleTransmission</type>
+      <joint name="gimbal${child3}">
+        <hardwareInterface>hardware_interface/EffortJointInterface</hardwareInterface>
+      </joint>
+      <actuator name="servo${child3}">
+        <hardwareInterface>hardware_interface/EffortJointInterface</hardwareInterface>
+        <mechanicalReduction>1</mechanicalReduction>
+      </actuator>
+    </transmission>
+    <transmission name="joint_tran${child4}">
+      <type>transmission_interface/SimpleTransmission</type>
+      <joint name="gimbal${child4}">
+        <hardwareInterface>hardware_interface/EffortJointInterface</hardwareInterface>
+      </joint>
+      <actuator name="servo${child4}">
+        <hardwareInterface>hardware_interface/EffortJointInterface</hardwareInterface>
+        <mechanicalReduction>1</mechanicalReduction>
+      </actuator>
+    </transmission>
+  </xacro:macro>
+  <xacro:macro name="rolling_thrust_link" params="self rotor_direction">
+    <link name="gimbal_link${self}">
+      <inertial>
+        <origin xyz="0 0 0" rpy="0 0 0"/>
+        <mass value="0.00001"/>
+        <inertia
+            ixx="0.000001" ixy="0.0" ixz="0.0"
+            iyy="0.000001" iyz="0.0"
+            izz="0.000001"/>
+      </inertial>
+      <visual>
+        <origin xyz="0 0 0" rpy="0 0 0" />
+        <geometry>
+          <cylinder radius="0.2" length="0.05" />
+        </geometry>
+      </visual>
+    </link>
+    ## rotor parent link (virtual)
+    <link name="rotor_parent${self}">
+      <inertial>
+        <origin xyz="0 0 0" rpy="0 0 0"/>
+        <mass value="0.00001"/>
+        <inertia
+            ixx="0.000001" ixy="0.0" ixz="0.0"
+            iyy="0.000001" iyz="0.0"
+            izz="0.000001"/>
+      </inertial>
+    </link>
+    ## thrust link (virtual)
+    <link name="thrust${self}">
+      <inertial>
+        <origin xyz="0 0 0" rpy="0 0 0"/>
+        <mass value="0.00001"/>
+        <inertia
+            ixx="0.001" ixy="0.0" ixz="0.0"
+            iyy="0.001" iyz="0.0"
+            izz="0.001"/>
+      </inertial>
+    </link>
+    #### joints ####
+    #### rotor parent link joint (virtual) ####
+    <joint name="rotor_parent_link_joint${self}" type="fixed">
+      <parent link="gimbal_link${self}"/>
+      <child link="rotor_parent${self}"/>
+      <origin rpy="0 0 0" xyz="0 0 0"/>
+      <axis xyz="0 0 1"/>
+    </joint>
+    #### rotor joint (virtual) ####
+    <joint name="rotor${self}" type="continuous">
+      <limit effort="100.0" lower="${min_force}" upper="${max_force}" velocity="0.5"/>
+      <parent link="rotor_parent${self}"/>
+      <child link="thrust${self}"/>
+      <origin rpy="0 0 0" xyz="0 0 0"/>
+      <axis xyz="0 0 ${rotor_direction}"/>
+    </joint>
+    <transmission name="rotor_tran${self}">
+      <type>transmission_interface/SimpleTransmission</type>
+      <joint name="rotor${self}">
+        <hardwareInterface>RotorInterface</hardwareInterface>
+      </joint>
+      <actuator name="rotor_actuator${self}">
+        <hardwareInterface>RotorInterface</hardwareInterface>
+        <mechanicalReduction>1</mechanicalReduction>
+      </actuator>
+    </transmission>
   </xacro:macro>
 </robot>

Commit message: [rolling] update model for 6 rotors

File: robots/rolling/robots/rolling.urdf.xacro (robot description, xacro)
@@ -4,8 +4,10 @@
   <xacro:include filename="$(find rolling)/urdf/rolling_link.urdf.xacro" />
   <xacro:include filename="$(find rolling)/urdf/common.xacro" />
-  <xacro:rolling_base_link child1="1" child2="2" child3="3" child4="4" />
+  <xacro:rolling_base_link child1="1" child2="2" child3="3" child4="4" child5="5" child6="6"/>
   <xacro:rolling_thrust_link self="1" rotor_direction="1" />
   <xacro:rolling_thrust_link self="2" rotor_direction="-1"/>
   <xacro:rolling_thrust_link self="3" rotor_direction="1"/>
   <xacro:rolling_thrust_link self="4" rotor_direction="-1"/>
+  <xacro:rolling_thrust_link self="5" rotor_direction="1"/>
+  <xacro:rolling_thrust_link self="6" rotor_direction="-1"/>
 </robot>

File: robots/rolling/urdf/common.xacro (robot description, xacro)
@@ -7,5 +7,5 @@
   <m_f_rate value="-0.0172" /> <!-- drug torque rate -->
   <xacro:property name="max_force" value="18.0" /> <!-- [N] -->
-  <xacro:property name="min_force" value="1.0" /> <!-- [N] -->
+  <xacro:property name="min_force" value="-18.0" /> <!-- [N] -->
   <!-- friction -->
   <xacro:macro name="friction" params="link">

File: robots/rolling/urdf/rolling_link.urdf.xacro (robot description, xacro)
@@ -3,5 +3,5 @@
     xmlns:xacro="http://www.ros.org/wiki/xacro" name="rolling_link" >
   <xacro:property name="cylinder_radius" value="1.0"/>
-  <xacro:macro name="rolling_base_link" params="child1 child2 child3 child4">
+  <xacro:macro name="rolling_base_link" params="child1 child2 child3 child4 child5 child6">
     <link name="root">
       <inertial>
@@ -26,5 +26,5 @@
         <mass value="1.0"/>
         <inertia
-            ixx="0.01" iyy="0.01" izz="0.01"
+            ixx="${0.5 * 1.0 * cylinder_radius * cylinder_radius}" iyy="${0.5 * 1.0 * cylinder_radius * cylinder_radius}" izz="${0.25 * 1.0 * cylinder_radius * cylinder_radius}"
             ixy="0.00001" ixz="0.00001" iyz="0.00001"/>
       </inertial>
@@ -70,9 +70,9 @@
       <dynamics damping="0.8" friction="0.0"/>
     </joint>
-  <joint name="gimbal${child2}" type="revolute">
+    <joint name="gimbal${child2}" type="revolute">
       <limit effort="6.6" lower="-1.57" upper="1.57" velocity="3.0"/>
       <parent link="base_link"/>
       <child link="gimbal_link${child2}"/>
-      <origin rpy="0 0 0" xyz="0 0 ${cylinder_radius - 0.2}"/>
+      <origin rpy="0 ${pi/2 -  pi/3 } 0" xyz="${(cylinder_radius - 0.2) * cos(pi / 3)} 0 ${(cylinder_radius - 0.2) * sin(pi / 3)}"/>
       <axis xyz="1 0 0"/>
       <dynamics damping="0.8" friction="0.0"/>
@@ -82,5 +82,5 @@
       <parent link="base_link"/>
       <child link="gimbal_link${child3}"/>
-      <origin rpy="0 ${-pi/2} 0" xyz="${- cylinder_radius + 0.2} 0 0"/>
+      <origin rpy="0 ${pi/2 - pi / 3 * 2} 0" xyz="${(cylinder_radius - 0.2) * cos(pi / 3 * 2)} 0 ${(cylinder_radius - 0.2) * sin(pi / 3 * 2)}"/>
       <axis xyz="1 0 0"/>
       <dynamics damping="0.8" friction="0.0"/>
@@ -90,5 +90,21 @@
       <parent link="base_link"/>
       <child link="gimbal_link${child4}"/>
-      <origin rpy="0 ${pi} 0" xyz="0 0 ${- cylinder_radius + 0.2}"/>
+      <origin rpy="0 ${pi/2 - pi / 3 * 3} 0" xyz="${(cylinder_radius - 0.2) * cos(pi / 3 * 3)} 0 ${(cylinder_radius - 0.2) * sin(pi / 3 * 3)}"/>
+      <axis xyz="1 0 0"/>
+      <dynamics damping="0.8" friction="0.0"/>
+    </joint>
+    <joint name="gimbal${child5}" type="revolute">
+      <limit effort="6.6" lower="-1.57" upper="1.57" velocity="3.0"/>
+      <parent link="base_link"/>
+      <child link="gimbal_link${child5}"/>
+      <origin rpy="0 ${pi/2 - pi / 3 * 4} 0" xyz="${(cylinder_radius - 0.2) * cos(pi / 3 * 4)} 0 ${(cylinder_radius - 0.2) * sin(pi / 3 * 4)}"/>
+      <axis xyz="1 0 0"/>
+      <dynamics damping="0.8" friction="0.0"/>
+    </joint>
+    <joint name="gimbal${child6}" type="revolute">
+      <limit effort="6.6" lower="-1.57" upper="1.57" velocity="3.0"/>
+      <parent link="base_link"/>
+      <child link="gimbal_link${child6}"/>
+      <origin rpy="0 ${pi/2 - pi / 3 * 5} 0" xyz="${(cylinder_radius - 0.2) * cos(pi / 3 * 5)} 0 ${(cylinder_radius - 0.2) * sin(pi / 3 * 5)}"/>
       <axis xyz="1 0 0"/>
       <dynamics damping="0.8" friction="0.0"/>
@@ -131,4 +147,24 @@
       </joint>
       <actuator name="servo${child4}">
+        <hardwareInterface>hardware_interface/EffortJointInterface</hardwareInterface>
+        <mechanicalReduction>1</mechanicalReduction>
+      </actuator>
+    </transmission>
+    <transmission name="joint_tran${child5}">
+      <type>transmission_interface/SimpleTransmission</type>
+      <joint name="gimbal${child5}">
+        <hardwareInterface>hardware_interface/EffortJointInterface</hardwareInterface>
+      </joint>
+      <actuator name="servo${child5}">
+        <hardwareInterface>hardware_interface/EffortJointInterface</hardwareInterface>
+        <mechanicalReduction>1</mechanicalReduction>
+      </actuator>
+    </transmission>
+    <transmission name="joint_tran${child6}">
+      <type>transmission_interface/SimpleTransmission</type>
+      <joint name="gimbal${child6}">
+        <hardwareInterface>hardware_interface/EffortJointInterface</hardwareInterface>
+      </joint>
+      <actuator name="servo${child6}">
         <hardwareInterface>hardware_interface/EffortJointInterface</hardwareInterface>
         <mechanicalReduction>1</mechanicalReduction>
@@ -145,7 +181,7 @@
         <mass value="0.1"/>
         <inertia
-            ixx="0.001" ixy="0.0" ixz="0.0"
-            iyy="0.001" iyz="0.0"
-            izz="0.001"/>
+            ixx="${0.25 * 0.1 * 0.2 * 0.2}" ixy="0.0" ixz="0.0"
+            iyy="${0.25 * 0.1 * 0.2 * 0.2}" iyz="0.0"
+            izz="${0.5 * 0.1 * 0.2 * 0.2}"/>
       </inertial>
       <collision>
