Commit message: [rolling][urdf] update inertia of urdf and rviz_config

File: robots/rolling/urdf/rolling_link.urdf.xacro (robot description, xacro)
@@ -26,5 +26,5 @@
         <mass value="1.0"/>
         <inertia
-            ixx="0.00001" iyy="0.00001" izz="0.00001"
+            ixx="0.01" iyy="0.01" izz="0.01"
             ixy="0.00001" ixz="0.00001" iyz="0.00001"/>
       </inertial>
@@ -66,5 +66,5 @@
       <parent link="base_link"/>
       <child link="gimbal_link${child1}"/>
-      <origin rpy="0 ${pi/2} 0" xyz="${cylinder_radius} 0 0"/>
+      <origin rpy="0 ${pi/2} 0" xyz="${cylinder_radius - 0.2} 0 0"/>
       <axis xyz="1 0 0"/>
       <dynamics damping="0.8" friction="0.0"/>
@@ -74,5 +74,5 @@
       <parent link="base_link"/>
       <child link="gimbal_link${child2}"/>
-      <origin rpy="0 0 0" xyz="0 0 ${cylinder_radius}"/>
+      <origin rpy="0 0 0" xyz="0 0 ${cylinder_radius - 0.2}"/>
       <axis xyz="1 0 0"/>
       <dynamics damping="0.8" friction="0.0"/>
@@ -82,5 +82,5 @@
       <parent link="base_link"/>
       <child link="gimbal_link${child3}"/>
-      <origin rpy="0 ${-pi/2} 0" xyz="${- cylinder_radius} 0 0"/>
+      <origin rpy="0 ${-pi/2} 0" xyz="${- cylinder_radius + 0.2} 0 0"/>
       <axis xyz="1 0 0"/>
       <dynamics damping="0.8" friction="0.0"/>
@@ -90,5 +90,5 @@
       <parent link="base_link"/>
       <child link="gimbal_link${child4}"/>
-      <origin rpy="0 ${pi} 0" xyz="0 0 ${- cylinder_radius}"/>
+      <origin rpy="0 ${pi} 0" xyz="0 0 ${- cylinder_radius + 0.2}"/>
       <axis xyz="1 0 0"/>
       <dynamics damping="0.8" friction="0.0"/>
@@ -135,7 +135,33 @@
       </actuator>
     </transmission>
+    <xacro:friction link="base_link"/>
   </xacro:macro>
   <xacro:macro name="rolling_thrust_link" params="self rotor_direction">
+    ## link
+    #### rotor parent link (virtual) ####
     <link name="gimbal_link${self}">
+      <inertial>
+        <origin xyz="0 0 0" rpy="0 0 0"/>
+        <mass value="0.1"/>
+        <inertia
+            ixx="0.001" ixy="0.0" ixz="0.0"
+            iyy="0.001" iyz="0.0"
+            izz="0.001"/>
+      </inertial>
+      <collision>
+        <origin xyz="0 0 0" rpy="0 0 0" />
+        <geometry>
+          <cylinder radius="0.2" length="0.05"/>
+        </geometry>
+      </collision>
+      <visual>
+        <origin xyz="0 0 0" rpy="0 0 0" />
+        <geometry>
+          <cylinder radius="0.2" length="0.05" />
+        </geometry>
+      </visual>
+    </link>
+    ## rotor parent link (virtual)
+    <link name="rotor_parent${self}">
       <inertial>
         <origin xyz="0 0 0" rpy="0 0 0"/>
@@ -146,21 +172,4 @@
             izz="0.000001"/>
       </inertial>
-      <visual>
-        <origin xyz="0 0 0" rpy="0 0 0" />
-        <geometry>
-          <cylinder radius="0.2" length="0.05" />
-        </geometry>
-      </visual>
-    </link>
-    ## rotor parent link (virtual)
-    <link name="rotor_parent${self}">
-      <inertial>
-        <origin xyz="0 0 0" rpy="0 0 0"/>
-        <mass value="0.00001"/>
-        <inertia
-            ixx="0.000001" ixy="0.0" ixz="0.0"
-            iyy="0.000001" iyz="0.0"
-            izz="0.000001"/>
-      </inertial>
     </link>
     ## thrust link (virtual)
@@ -175,4 +184,5 @@
       </inertial>
     </link>
+    <xacro:damping_factor link="thrust${self}" />
     #### joints ####
     #### rotor parent link joint (virtual) ####
@@ -181,5 +191,5 @@
       <child link="rotor_parent${self}"/>
       <origin rpy="0 0 0" xyz="0 0 0"/>
-      <axis xyz="0 0 1"/>
+      <axis xyz="0 0 ${rotor_direction}"/>
     </joint>
     #### rotor joint (virtual) ####

Commit message: [rolling][urdf] add rotor neutral coordinates in urdf

File: robots/rolling/urdf/rolling_link.urdf.xacro (robot description, xacro)
@@ -3,4 +3,5 @@
     xmlns:xacro="http://www.ros.org/wiki/xacro" name="rolling_link" >
   <xacro:property name="rotor_offset" value="0.05" />
+  <xacro:property name="rotor_tilt" value="0.2" />
   <xacro:macro name="rolling_module" params="self child baselink rotor_direction">
     ### link ###
@@ -76,5 +77,5 @@
       </inertial>
       <visual>
-        <origin rpy="0 ${(self % 2 * 2 - 1) * 0.2} 0" xyz="0 0 0"/>
+        <origin rpy="0 ${(self % 2 * 2 - 1) * rotor_tilt} 0" xyz="0 0 0"/>
         <geometry>
           <mesh filename="package://rolling/urdf/mesh/roll_gimbal_module.dae" />
@@ -105,10 +106,10 @@
       <parent link="link${self}"/>
       <child link="gimbal_link${self}"/>
-      <origin xyz="0.3 0 0" rpy="0 ${((self % 2) * 2 - 1) * 0.2} 0" />
+      <origin xyz="0.3 0 0" rpy="0 0 0" />
       <axis xyz="1 0 0"/>
       <dynamics damping="0.1" friction="0.0"/>
     </joint>
-    #### rotor parent link (virtual) ####
-    <link name="rotor_parent${self}">
+    #### rotor coord link (virtual) ####
+    <link name="rotor_coord${self}">
       <inertial>
         <origin xyz="0 0 0" rpy="0 0 0"/>
@@ -120,6 +121,6 @@
       </inertial>
     </link>
-    #### thrust link (virtual) ####
-    <link name="thrust${self}">
+    #### rotor parent link (virtual) ####
+    <link name="rotor_parent${self}">
       <inertial>
         <origin xyz="0 0 0" rpy="0 0 0"/>
@@ -131,10 +132,28 @@
       </inertial>
     </link>
+    #### thrust link (virtual) ####
+    <link name="thrust${self}">
+      <inertial>
+        <origin xyz="0 0 0" rpy="0 0 0"/>
+        <mass value="0.00001"/>
+        <inertia
+            ixx="0.000001" ixy="0.0" ixz="0.0"
+            iyy="0.000001" iyz="0.0"
+            izz="0.000001"/>
+      </inertial>
+    </link>
     <xacro:damping_factor link="thrust${self}" />
+    #### rotor coord link joint (virtual) ####
+    <joint name="rotor_coord_link_joint${self}" type="fixed">
+      <parent link="link${self}"/>
+      <child link="rotor_coord${self}"/>
+      <origin rpy="0 ${(self % 2 * 2 - 1) * rotor_tilt} 0" xyz="0.3 0 0"/>
+      <axis xyz="0 0 1"/>
+    </joint>
     #### rotor parent link joint (virtual) ####
     <joint name="rotor_parent_link_joint${self}" type="fixed">
       <parent link="gimbal_link${self}"/>
       <child link="rotor_parent${self}"/>
-      <origin rpy="0 0 0" xyz="0 0 ${rotor_offset}"/> # TODO: update rotor position
+      <origin rpy="0 ${(self % 2 * 2 - 1) * rotor_tilt} 0" xyz="0 0 ${rotor_offset}"/> # TODO: update rotor position
       <axis xyz="0 0 1"/>
     </joint>
