Commit message: [rolling] refactored urdf directory

File: robots/rolling/urdf/common.xacro (robot description, xacro)
@@ -20,3 +20,13 @@
     </gazebo>
   </xacro:macro>
+  <xacro:macro name="glay">
+    <material name="glay" >
+      <color rgba="0.5 0.5 0.5 1.0" />
+    </material>
+  </xacro:macro>
+  <xacro:macro name="black">
+    <material name="black" >
+      <color rgba="0 0 0 1.0" />
+    </material>
+  </xacro:macro>
 </robot>

Commit message: [rolling][urdf] update urdf

File: robots/rolling/urdf/common.xacro (robot description, xacro)
@@ -13,4 +13,11 @@
       <mu1>0.4</mu1>
       <mu2>0.4</mu2>
+    </gazebo>
+  </xacro:macro>
+  <!-- large friction -->
+  <xacro:macro name="large_friction" params="link">
+    <gazebo reference="${link}">
+      <mu1>1.5</mu1>
+      <mu2>1.5</mu2>
     </gazebo>
   </xacro:macro>

File: robots/rolling/urdf/shelled/rolling_link.urdf.xacro (robot description, xacro)
@@ -21,10 +21,10 @@
         <xacro:glay/>
       </visual>
-      <collision>
-        <origin xyz="0.225 0 0" rpy="0 0 0" />
-        <geometry>
-          <box size="0.6135 0.052 0.15" />
-        </geometry>
-      </collision>
+      <!-- <collision> -->
+      <!--   <origin xyz="0.225 0 0" rpy="0 0 0" /> -->
+      <!--   <geometry> -->
+      <!--     <box size="0.6135 0.052 0.15" /> -->
+      <!--   </geometry> -->
+      <!-- </collision> -->
     </link>
     ### link${self} ###
@@ -72,5 +72,5 @@
         <axis xyz="0 0 1"/>
       </joint>
-      <xacro:friction link="cylinder_collision"/>
+      <xacro:large_friction link="cylinder_collision"/>
     </xacro:if>
     <!-- set the fcu frame -->

Commit message: [rolling][urdf] modify maximum thrust

File: robots/rolling/urdf/common.xacro (robot description, xacro)
@@ -6,5 +6,5 @@
   <thrust_link name="thrust" />
   <m_f_rate value="-0.0142" /> <!-- drug torque rate -->
-  <xacro:property name="max_force" value="18.0" /> <!-- [N] -->
+  <xacro:property name="max_force" value="22.0" /> <!-- [N] -->
   <xacro:property name="min_force" value="0.0" /> <!-- [N] -->
   <!-- friction -->
