Commit message: [rolling][OptimalDesign][WIP] add optimization node

File: robots/rolling/urdf/shelled_opt/rolling_link_opt.urdf.xacro (robot description, xacro)
@@ -130,5 +130,5 @@
     #### gimbal joint ####
     <joint name="gimbal${self}" type="continuous" >
-      <limit effort="3" lower="-3.14" upper="3.14" velocity="12.5"/>
+      <limit effort="10" lower="-3.14" upper="3.14" velocity="12.5"/>
       <parent link="link${self}"/>
       <child link="gimbal_link${self}"/>
@@ -149,4 +149,14 @@
     </link>
     #### rotor parent link (virtual) ####
+    <link name="rotor_parent_parent${self}">
+      <inertial>
+        <origin xyz="0 0 0" rpy="0 0 0"/>
+        <mass value="0.00001"/>
+        <inertia
+            ixx="0.0001" ixy="0.0" ixz="0.0"
+            iyy="0.0001" iyz="0.0"
+            izz="0.0002"/>
+      </inertial>
+    </link>
     <link name="rotor_parent${self}">
       <inertial>
@@ -181,9 +191,16 @@
     </joint>
     #### rotor parent link joint (virtual) ####
-    <joint name="gimbal_parent${self}" type="continuous">
-      <limit effort="3.0" lower="${-pi/2}" upper="${pi/2}" velocity="12.5"/>
+    <joint name="gimbal_parent_parent${self}" type="fixed">
       <parent link="gimbal_link${self}"/>
+      <child link="rotor_parent_parent${self}"/>
+      <origin rpy="0 0 0" xyz="0 0 ${rotor_offset}"/> # TODO: update rotor position
+      <axis xyz="0 1 0"/>
+      <dynamics damping="0.1" friction="0.0"/>
+    </joint>
+    <joint name="gimbal_pitch${self}" type="continuous">
+      <limit effort="10.0" lower="${-pi/2}" upper="${pi/2}" velocity="12.5"/>
+      <parent link="rotor_parent_parent${self}"/>
       <child link="rotor_parent${self}"/>
-      <origin rpy="0 0 0" xyz="0 0 ${rotor_offset}"/> # TODO: update rotor position
+      <origin rpy="0 0 0" xyz="0 0 0"/> # TODO: update rotor position
       <axis xyz="0 1 0"/>
       <dynamics damping="0.1" friction="0.0"/>
@@ -220,14 +237,4 @@
       </actuator>
     </transmission>
-    <transmission name="gimbal_parent_tran${self}">
-      <type>transmission_interface/SimpleTransmission</type>
-      <joint name="gimbal_parent${self}">
-        <hardwareInterface>hardware_interface/EffortJointInterface</hardwareInterface>
-      </joint>
-      <actuator name="gimbal_parent${self}">
-        <hardwareInterface>hardware_interface/EffortJointInterface</hardwareInterface>
-        <mechanicalReduction>1</mechanicalReduction>
-      </actuator>
-    </transmission>
     <transmission name="gimbal_tran${self}">
       <type>transmission_interface/SimpleTransmission</type>
@@ -236,4 +243,14 @@
       </joint>
       <actuator name="gimbal_servo${self}">
+        <hardwareInterface>hardware_interface/EffortJointInterface</hardwareInterface>
+        <mechanicalReduction>1</mechanicalReduction>
+      </actuator>
+    </transmission>
+    <transmission name="gimbal_pitch_tran${self}">
+      <type>transmission_interface/SimpleTransmission</type>
+      <joint name="gimbal_pitch${self}">
+        <hardwareInterface>hardware_interface/EffortJointInterface</hardwareInterface>
+      </joint>
+      <actuator name="gimbal_pitch_servo${self}">
         <hardwareInterface>hardware_interface/EffortJointInterface</hardwareInterface>
         <mechanicalReduction>1</mechanicalReduction>
