Commit message: [rolling] update urdf for collision

File: robots/rolling/urdf/shelled/rolling_link.urdf.xacro (robot description, xacro)
@@ -49,4 +49,29 @@
       </joint>
     </xacro:if>
+    <!-- cylinder collision model  -->
+    <xacro:if value="${baselink}">
+      <link name="cylinder_collision">
+        <inertial>
+          <origin xyz="0 0 0" rpy="0 0 0"/>
+          <mass value="0.00001"/>
+          <inertia
+              ixx="0.000001" ixy="0.0" ixz="0.0"
+              iyy="0.000001" iyz="0.0"
+              izz="0.000001"/>
+        </inertial>
+        <collision>
+          <geometry>
+            <cylinder radius="0.4" length="0.03"/>
+          </geometry>
+        </collision>
+      </link>
+      <joint name="cylinder_collision_joint" type="fixed">
+        <parent link="link${self}"/>
+        <child link="cylinder_collision"/>
+        <origin rpy="0 0 0" xyz="0.262 0.153 0"/>
+        <axis xyz="0 0 1"/>
+      </joint>
+      <xacro:friction link="cylinder_collision"/>
+    </xacro:if>
     <!-- set the fcu frame -->
     <xacro:if value="${baselink}">
@@ -85,7 +110,7 @@
       </visual>
       <collision>
-        <origin xyz="0 0 ${rotor_offset}" />
-        <geometry>
-          <cylinder radius="0.2" length="0.05" />
+        <origin xyz="0 0 ${rotor_offset}" rpy="0 ${(self % 2 * 2 - 1) * rotor_tilt} 0" />
+        <geometry>
+          <cylinder radius="0.1" length="0.05" />
         </geometry>
       </collision>

Commit message: [rolling] enable to set tilt of rotor as parameter

File: robots/rolling/urdf/shelled/rolling_link.urdf.xacro (robot description, xacro)
@@ -3,5 +3,7 @@
     xmlns:xacro="http://www.ros.org/wiki/xacro" name="rolling_link" >
   <xacro:property name="rotor_offset" value="0.05" />
-  <xacro:property name="rotor_tilt" value="0.1" />
+  <xacro:property name="rotor1_tilt" value="0.0" />
+  <xacro:property name="rotor2_tilt" value="0.0" />
+  <xacro:property name="rotor3_tilt" value="0.0" />
   <xacro:macro name="rolling_module" params="self child baselink rotor_direction">
     ### link ###
@@ -103,5 +105,13 @@
       </inertial>
       <visual>
-        <origin rpy="0 ${(self % 2 * 2 - 1) * rotor_tilt} 0" xyz="0 0 0"/>
+        <xacro:if value="${self == 1}">
+          <origin rpy="0 ${rotor1_tilt} 0" xyz="0 0 0"/>
+        </xacro:if>
+        <xacro:if value="${self == 2}">
+          <origin rpy="0 ${rotor2_tilt} 0" xyz="0 0 0"/>
+        </xacro:if>
+        <xacro:if value="${self == 3}">
+          <origin rpy="0 ${rotor3_tilt} 0" xyz="0 0 0"/>
+        </xacro:if>
         <geometry>
           <mesh filename="package://rolling/urdf/shelled/mesh/roll_gimbal_module.STL" scale="0.001 0.001 0.001"/>
@@ -110,5 +120,13 @@
       </visual>
       <collision>
-        <origin xyz="0 0 ${rotor_offset}" rpy="0 ${(self % 2 * 2 - 1) * rotor_tilt} 0" />
+        <xacro:if value="${self == 1}">
+          <origin xyz="0 0 ${rotor_offset}" rpy="0 ${rotor1_tilt} 0" />
+        </xacro:if>
+        <xacro:if value="${self == 2}">
+          <origin xyz="0 0 ${rotor_offset}" rpy="0 ${rotor2_tilt} 0" />
+        </xacro:if>
+        <xacro:if value="${self == 3}">
+          <origin xyz="0 0 ${rotor_offset}" rpy="0 ${rotor3_tilt} 0" />
+        </xacro:if>
         <geometry>
           <cylinder radius="0.1" length="0.05" />
@@ -175,6 +193,14 @@
       <parent link="link${self}"/>
       <child link="rotor_coord${self}"/>
-      <origin rpy="0 ${(self % 2 * 2 - 1) * rotor_tilt} 0" xyz="0.3 0 0"/>
-      <axis xyz="0 0 1"/>
+      <xacro:if value="${self == 1}">
+        <origin rpy="0 ${rotor1_tilt} 0" xyz="0.3 0 0"/>
+      </xacro:if>
+      <xacro:if value="${self == 2}">
+        <origin rpy="0 ${rotor2_tilt} 0" xyz="0.3 0 0"/>
+      </xacro:if>
+      <xacro:if value="${self == 3}">
+        <origin rpy="0 ${rotor3_tilt} 0" xyz="0.3 0 0"/>
+      </xacro:if>
+        <axis xyz="0 0 1"/>
     </joint>
     #### rotor parent link joint (virtual) ####
@@ -182,5 +208,13 @@
       <parent link="gimbal_link${self}"/>
       <child link="rotor_parent${self}"/>
-      <origin rpy="0 ${(self % 2 * 2 - 1) * rotor_tilt} 0" xyz="0 0 ${rotor_offset}"/> # TODO: update rotor position
+      <xacro:if value="${self == 1}">
+        <origin rpy="0 ${rotor1_tilt} 0" xyz="0 0 ${rotor_offset}"/> # TODO: update rotor position
+      </xacro:if>
+      <xacro:if value="${self == 2}">
+        <origin rpy="0 ${rotor2_tilt} 0" xyz="0 0 ${rotor_offset}"/> # TODO: update rotor position
+      </xacro:if>
+      <xacro:if value="${self == 3}">
+        <origin rpy="0 ${rotor3_tilt} 0" xyz="0 0 ${rotor_offset}"/> # TODO: update rotor position
+      </xacro:if>
       <axis xyz="0 0 1"/>
     </joint>

Commit message: [rolling][urdf] add dae

File: robots/rolling/urdf/shelled/rolling_link.urdf.xacro (robot description, xacro)
@@ -19,5 +19,5 @@
         <origin rpy="0 0 0" xyz="0 0 0"/>
         <geometry>
-          <mesh filename="package://rolling/urdf/shelled/mesh/link.STL" scale="0.001 0.001 0.001"/>
+          <mesh filename="package://rolling/urdf/shelled/mesh/link.dae" scale="0.001 0.001 0.001"/>
         </geometry>
         <xacro:glay/>
@@ -115,5 +115,5 @@
         </xacro:if>
         <geometry>
-          <mesh filename="package://rolling/urdf/shelled/mesh/roll_gimbal_module.STL" scale="0.001 0.001 0.001"/>
+          <mesh filename="package://rolling/urdf/shelled/mesh/roll_gimbal_module.dae" scale="0.001 0.001 0.001"/>
         </geometry>
         <xacro:black/>

Commit message: [rolling] update rotor tilt

File: robots/rolling/urdf/shelled/rolling_link.urdf.xacro (robot description, xacro)
@@ -3,7 +3,7 @@
     xmlns:xacro="http://www.ros.org/wiki/xacro" name="rolling_link" >
   <xacro:property name="rotor_offset" value="0.05" />
-  <xacro:property name="rotor1_tilt" value="0.0" />
-  <xacro:property name="rotor2_tilt" value="0.0" />
-  <xacro:property name="rotor3_tilt" value="0.0" />
+  <xacro:property name="rotor1_tilt" value="-0.125" />
+  <xacro:property name="rotor2_tilt" value="0.146" />
+  <xacro:property name="rotor3_tilt" value="0.083" />
   <xacro:macro name="rolling_module" params="self child baselink rotor_direction">
     ### link ###
@@ -64,5 +64,5 @@
         <collision>
           <geometry>
-            <cylinder radius="0.4" length="0.03"/>
+            <cylinder radius="0.4" length="0.23"/>
           </geometry>
         </collision>
@@ -106,11 +106,11 @@
       <visual>
         <xacro:if value="${self == 1}">
-          <origin rpy="0 ${rotor1_tilt} 0" xyz="0 0 0"/>
+          <origin rpy="0 0 0" xyz="0 0 0"/>
         </xacro:if>
         <xacro:if value="${self == 2}">
-          <origin rpy="0 ${rotor2_tilt} 0" xyz="0 0 0"/>
+          <origin rpy="0 0 0" xyz="0 0 0"/>
         </xacro:if>
         <xacro:if value="${self == 3}">
-          <origin rpy="0 ${rotor3_tilt} 0" xyz="0 0 0"/>
+          <origin rpy="0 0 0" xyz="0 0 0"/>
         </xacro:if>
         <geometry>
