Commit message: [rolling][control][WIP] not use rotor refine process and separate wrench allocation process for under actuated control. add sr-inverse option for wrench allocation

File: robots/rolling/robots/20230808_frameless/rolling.urdf.xacro (robot description, xacro)
@@ -6,4 +6,4 @@
   <xacro:rolling_module self="1" child="2" rotor_direction="1"  battery="false"/>
   <xacro:rolling_module self="2" child="3" rotor_direction="-1" battery="false"/>
-  <xacro:rolling_module self="3" child="3" rotor_direction="1"  battery="false"/>
+  <xacro:rolling_module self="3" child="3" rotor_direction="1"  battery="true"/>
 </robot>

File: robots/rolling/urdf/20230808_frameless/rolling_link.urdf.xacro (robot description, xacro)
@@ -120,11 +120,11 @@
       <axis xyz="0 0 1"/>
       <xacro:if value="${self == 1}">
-        <origin xyz="-0.00586 0 0.08439" rpy="0 -0.125 0"/>
+        <origin xyz="0 0 0" rpy="0 -0.125 0"/>
       </xacro:if>
       <xacro:if value="${self == 2}">
-        <origin xyz="0.01037 0 0.0846" rpy="0 0.146 0"/>
+        <origin xyz="0 0 0" rpy="0 0.146 0"/>
       </xacro:if>
       <xacro:if value="${self == 3}">
-        <origin xyz="0.00389 0 0.08417" rpy="0 0.083 0"/>
+        <origin xyz="0 0 0" rpy="0 0.083 0"/>
       </xacro:if>
     </joint>
