Commit message: [rolling] update urdf

File: robots/rolling/urdf/20230808_frameless/link1.urdf.xacro (robot description, xacro)
@@ -5,9 +5,9 @@
     <link name="link1">
       <inertial>
-        <origin xyz="0.31793422 -0.00000349 0.01201593" rpy="0 0 0"/>
-        <mass value="0.32946729"/>
+        <origin xyz="0.26695257 0.00000500 0.00993736" rpy="0 0 0"/>
+        <mass value="0.48484449"/>
         <inertia
-            ixx="0.00046940" iyy="0.01038614" izz="0.01000885"
-            ixy="0.00000061" ixz="0.00127450" iyz="0.00000002"/>
+            ixx="0.00050326"  iyy="0.01670962" izz="0.01633157"
+            ixy="-0.00000023" ixz="0.00133774" iyz="0.00000004"/>
       </inertial>
       <visual>
@@ -25,9 +25,9 @@
     <link name="gimbal_link1">
       <inertial>
-        <origin xyz="0.00711095 -0.00001676 0.02365341" rpy="0 0 0"/>
-        <mass value="0.29635001"/>
+        <origin xyz="0.00721656 -0.00001666 0.02317238" rpy="0 0 0"/>
+        <mass value="0.29811001"/>
         <inertia
-            ixx="0.00093502"  iyy="0.00101745"  izz="0.00023393"
-            ixy="-0.00000003" ixz="-0.00022207" iyz="0.00000025"/>
+            ixx="0.00094718"  iyy="0.00102969"  izz="0.00023510"
+            ixy="-0.00000002" ixz="-0.00022462" iyz="0.00000024"/>
       </inertial>
       <visual>

File: robots/rolling/urdf/20230808_frameless/link2.urdf.xacro (robot description, xacro)
@@ -5,9 +5,9 @@
     <link name="link2">
       <inertial>
-        <origin xyz="0.26329859 -0.00016231 0.00746546" rpy="0 0 0"/>
-        <mass value="0.50417254"/>
+        <origin xyz="0.26724120 -0.00000341 0.00917818" rpy="0 0 0"/>
+        <mass value="0.55395179"/>
         <inertia
-            ixx="0.00065269" iyy="0.01910297" izz="0.01867466"
-            ixy="0.00001175" ixz="0.00180333" iyz="0.00000367"/>
+            ixx="0.00055160"  iyy="0.02080064" izz="0.02042362"
+            ixy="-0.00000055" ixz="0.00153902" iyz="-0.00000007"/>
       </inertial>
       <visual>
@@ -25,9 +25,9 @@
     <link name="gimbal_link2">
       <inertial>
-        <origin xyz="0.01274450 -0.00001684 0.02393903" rpy="0 0 0"/>
-        <mass value="0.29654765"/>
+        <origin xyz="0.01281681 -0.00001674 0.02345664" rpy="0 0 0"/>
+        <mass value="0.29830765"/>
         <inertia
-            ixx="0.00094271" iyy="0.00099628" izz="0.00020518"
-            ixy="0.00000000" ixz="-0.00015385" iyz="0.00000025"/>
+            ixx="0.00095496" iyy="0.00100830"  izz="0.00020605"
+            ixy="0.00000000" ixz="-0.00015560" iyz="0.00000025"/>
       </inertial>
       <visual>

File: robots/rolling/urdf/20230808_frameless/link3.urdf.xacro (robot description, xacro)
@@ -5,9 +5,9 @@
     <link name="link3">
       <inertial>
-        <origin xyz="0.23026123 0.00000000 -0.01668659" rpy="0 0 0"/>
-        <mass value="0.22538003"/>
+        <origin xyz="0.21323824 0.00000000 -0.00885891" rpy="0 0 0"/>
+        <mass value="0.34751322"/>
         <inertia
-            ixx="0.00035669" iyy="0.00886443"  izz="0.00860000"
-            ixy="0.00000000" ixz="-0.00009841" iyz="0.00000000"/>
+            ixx="0.00041721" iyy="0.01179645"  izz="0.01149579"
+            ixy="0.00000000" ixz="-0.00026812" iyz="0.00000000"/>
       </inertial>
       <visual>
@@ -25,9 +25,9 @@
     <link name="gimbal_link3">
       <inertial>
-        <origin xyz="0.01050287 -0.00001677 0.02348758" rpy="0 0 0"/>
-        <mass value="0.29626563"/>
+        <origin xyz="0.01058848 -0.00001677 0.02300739" rpy="0 0 0"/>
+        <mass value="0.29802563"/>
         <inertia
-            ixx="0.00093068" iyy="0.00099429"  izz="0.00021506"
-            ixy="0.00000000" ixz="-0.00018040" iyz="0.00000025"/>
+            ixx="0.00094280" iyy="0.00100629"  izz="0.00021604"
+            ixy="0.00000000" ixz="-0.00018246" iyz="0.00000025"/>
       </inertial>
       <visual>

File: robots/rolling/urdf/20230808_frameless/rolling_link.urdf.xacro (robot description, xacro)
@@ -50,5 +50,5 @@
         <child link="fc" />
         <parent link="link${self}" />
-        <origin xyz="0.093 0.0012 0.0489" rpy="0 0 0" />
+        <origin xyz="0.0864 -0.0012 0.020" rpy="0 0 0" />
         <axis xyz="0 0 1"/>
       </joint>
