Commit message: [WIP][rolling] default rotor configuration (center of link, not tilted)

File: robots/rolling/urdf/20230808_frameless/rolling_link.urdf.xacro (robot description, xacro)
@@ -62,11 +62,14 @@
       <dynamics damping="0.1" friction="0.0"/>
       <xacro:if value="${self == 1}">
-        <origin xyz="0.170 0 0" rpy="0 0 0" />
+        <!-- <origin xyz="0.170 0 0" rpy="0 0 0" /> -->
+        <origin xyz="0.250 0 0" rpy="0 0 0" />
       </xacro:if>
       <xacro:if value="${self == 2}">
-        <origin xyz="0.2035 0 0" rpy="0 0 0" />
+        <!-- <origin xyz="0.2035 0 0" rpy="0 0 0" /> -->
+        <origin xyz="0.2835 0 0" rpy="0 0 0" />
       </xacro:if>
       <xacro:if value="${self == 3}">
-        <origin xyz="0.2035 0 0" rpy="0 0 0" />
+        <!-- <origin xyz="0.2035 0 0" rpy="0 0 0" /> -->
+        <origin xyz="0.2835 0 0" rpy="0 0 0" />
       </xacro:if>
     </joint>
@@ -120,11 +123,14 @@
       <axis xyz="0 0 1"/>
       <xacro:if value="${self == 1}">
-        <origin xyz="0 0 0" rpy="0 -0.125 0"/>
-      </xacro:if>
+        <!-- <origin xyz="0 0 0" rpy="0 -0.125 0"/> -->
+        <origin xyz="0 0 0" rpy="0 0 0"/>
+     </xacro:if>
       <xacro:if value="${self == 2}">
-        <origin xyz="0 0 0" rpy="0 0.146 0"/>
+        <!-- <origin xyz="0 0 0" rpy="0 0.146 0"/> -->
+        <origin xyz="0 0 0" rpy="0 0 0"/>
       </xacro:if>
       <xacro:if value="${self == 3}">
-        <origin xyz="0 0 0" rpy="0 0.083 0"/>
+        <!-- <origin xyz="0 0 0" rpy="0 0.083 0"/> -->
+        <origin xyz="0 0 0" rpy="0 0 0"/>
       </xacro:if>
     </joint>

Commit message: [rolling][urdf] add virtual link for cylinder collision model

File: robots/rolling/urdf/20230808_frameless/rolling_link.urdf.xacro (robot description, xacro)
@@ -106,4 +106,29 @@
         </xacro:if>
       </joint>
+    </xacro:if>
+    <!-- cylinder collision model  -->
+    <xacro:if value="${self == 2}">
+      <link name="cylinder_collision">
+        <inertial>
+          <origin xyz="0 0 0" rpy="0 0 0"/>
+          <mass value="0.00001"/>
+          <inertia
+              ixx="0.000001" ixy="0.0" ixz="0.0"
+              iyy="0.000001" iyz="0.0"
+              izz="0.000001"/>
+        </inertial>
+        <collision>
+          <geometry>
+            <cylinder radius="0.4" length="0.1"/>
+          </geometry>
+        </collision>
+      </link>
+      <joint name="cylinder_collision_joint" type="fixed">
+        <parent link="link${self}"/>
+        <child link="cylinder_collision"/>
+        <origin rpy="0 0 0" xyz="0.262 0.153 0"/>
+        <axis xyz="0 0 1"/>
+      </joint>
+      <xacro:large_friction link="cylinder_collision"/>
     </xacro:if>
     <!-- rotor parent (virtual) -->

File: robots/rolling/urdf/common.xacro (robot description, xacro)
@@ -18,6 +18,6 @@
   <xacro:macro name="large_friction" params="link">
     <gazebo reference="${link}">
-      <mu1>1.5</mu1>
-      <mu2>1.5</mu2>
+      <mu1>20</mu1>
+      <mu2>20</mu2>
     </gazebo>
   </xacro:macro>

File: robots/rolling/urdf/shelled/rolling_link.urdf.xacro (robot description, xacro)
@@ -64,5 +64,5 @@
         <collision>
           <geometry>
-            <cylinder radius="0.4" length="0.23"/>
+            <cylinder radius="0.4" length="0.1"/>
           </geometry>
         </collision>

Commit message: Revert "[WIP][rolling] default rotor configuration (center of link, not tilted)"
This reverts commit 43932c6294a85d3777902e46c92f17b3fa86c02c.

File: robots/rolling/urdf/20230808_frameless/rolling_link.urdf.xacro (robot description, xacro)
@@ -62,14 +62,11 @@
       <dynamics damping="0.1" friction="0.0"/>
       <xacro:if value="${self == 1}">
-        <!-- <origin xyz="0.170 0 0" rpy="0 0 0" /> -->
-        <origin xyz="0.250 0 0" rpy="0 0 0" />
+        <origin xyz="0.170 0 0" rpy="0 0 0" />
       </xacro:if>
       <xacro:if value="${self == 2}">
-        <!-- <origin xyz="0.2035 0 0" rpy="0 0 0" /> -->
-        <origin xyz="0.2835 0 0" rpy="0 0 0" />
+        <origin xyz="0.2035 0 0" rpy="0 0 0" />
       </xacro:if>
       <xacro:if value="${self == 3}">
-        <!-- <origin xyz="0.2035 0 0" rpy="0 0 0" /> -->
-        <origin xyz="0.2835 0 0" rpy="0 0 0" />
+        <origin xyz="0.2035 0 0" rpy="0 0 0" />
       </xacro:if>
     </joint>
@@ -148,14 +145,11 @@
       <axis xyz="0 0 1"/>
       <xacro:if value="${self == 1}">
-        <!-- <origin xyz="0 0 0" rpy="0 -0.125 0"/> -->
-        <origin xyz="0 0 0" rpy="0 0 0"/>
-     </xacro:if>
+        <origin xyz="0 0 0" rpy="0 -0.125 0"/>
+      </xacro:if>
       <xacro:if value="${self == 2}">
-        <!-- <origin xyz="0 0 0" rpy="0 0.146 0"/> -->
-        <origin xyz="0 0 0" rpy="0 0 0"/>
+        <origin xyz="0 0 0" rpy="0 0.146 0"/>
       </xacro:if>
       <xacro:if value="${self == 3}">
-        <!-- <origin xyz="0 0 0" rpy="0 0.083 0"/> -->
-        <origin xyz="0 0 0" rpy="0 0 0"/>
+        <origin xyz="0 0 0" rpy="0 0.083 0"/>
       </xacro:if>
     </joint>
