Commit message: [rolling][urdf] moved meshes

File: robots/rolling/urdf/20230808_frameless/battery.urdf.xacro (robot description, xacro)
@@ -13,5 +13,5 @@
       <visual>
         <geometry>
-          <mesh filename="package://rolling/urdf/20230808_frameless/mesh/battery_module.dae" scale="0.001 0.001 0.001"/>
+          <mesh filename="package://rolling/urdf/mesh/20230808_frameless/battery_module.dae" scale="0.001 0.001 0.001"/>
         </geometry>
       </visual>

File: robots/rolling/urdf/20230808_frameless/link1.urdf.xacro (robot description, xacro)
@@ -13,5 +13,5 @@
       <visual>
         <geometry>
-          <mesh filename="package://rolling/urdf/20230808_frameless/mesh/link1_base.dae" scale="0.001 0.001 0.001"/>
+          <mesh filename="package://rolling/urdf/mesh/20230808_frameless/link1_base.dae" scale="0.001 0.001 0.001"/>
         </geometry>
       </visual>
@@ -33,5 +33,5 @@
       <visual>
         <geometry>
-          <mesh filename="package://rolling/urdf/20230808_frameless/mesh/link1_gimbal.dae" scale="0.001 0.001 0.001"/>
+          <mesh filename="package://rolling/urdf/mesh/20230808_frameless/link1_gimbal.dae" scale="0.001 0.001 0.001"/>
         </geometry>
       </visual>

File: robots/rolling/urdf/20230808_frameless/link2.urdf.xacro (robot description, xacro)
@@ -13,5 +13,5 @@
       <visual>
         <geometry>
-          <mesh filename="package://rolling/urdf/20230808_frameless/mesh/link2_base.dae" scale="0.001 0.001 0.001"/>
+          <mesh filename="package://rolling/urdf/mesh/20230808_frameless/link2_base.dae" scale="0.001 0.001 0.001"/>
         </geometry>
       </visual>
@@ -33,5 +33,5 @@
       <visual>
         <geometry>
-          <mesh filename="package://rolling/urdf/20230808_frameless/mesh/link2_gimbal.dae" scale="0.001 0.001 0.001"/>
+          <mesh filename="package://rolling/urdf/mesh/20230808_frameless/link2_gimbal.dae" scale="0.001 0.001 0.001"/>
         </geometry>
       </visual>

File: robots/rolling/urdf/20230808_frameless/link3.urdf.xacro (robot description, xacro)
@@ -13,5 +13,5 @@
       <visual>
         <geometry>
-          <mesh filename="package://rolling/urdf/20230808_frameless/mesh/link3_base.dae" scale="0.001 0.001 0.001"/>
+          <mesh filename="package://rolling/urdf/mesh/20230808_frameless/link3_base.dae" scale="0.001 0.001 0.001"/>
         </geometry>
       </visual>
@@ -33,5 +33,5 @@
       <visual>
         <geometry>
-          <mesh filename="package://rolling/urdf/20230808_frameless/mesh/link3_gimbal.dae" scale="0.001 0.001 0.001"/>
+          <mesh filename="package://rolling/urdf/mesh/20230808_frameless/link3_gimbal.dae" scale="0.001 0.001 0.001"/>
         </geometry>
       </visual>

File: robots/rolling/urdf/shelled/rolling_link.urdf.xacro (robot description, xacro)
@@ -19,5 +19,5 @@
         <origin rpy="0 0 0" xyz="0 0 0"/>
         <geometry>
-          <mesh filename="package://rolling/urdf/shelled/mesh/link.dae" scale="0.001 0.001 0.001"/>
+          <mesh filename="package://rolling/urdf/mesh/shelled/link.dae" scale="0.001 0.001 0.001"/>
         </geometry>
         <xacro:glay/>
@@ -115,5 +115,5 @@
         </xacro:if>
         <geometry>
-          <mesh filename="package://rolling/urdf/shelled/mesh/roll_gimbal_module.dae" scale="0.001 0.001 0.001"/>
+          <mesh filename="package://rolling/urdf/mesh/shelled/roll_gimbal_module.dae" scale="0.001 0.001 0.001"/>
         </geometry>
         <xacro:black/>

Commit message: [rolling][urdf] changed mesh size to m unit

File: robots/rolling/urdf/20230808_frameless/battery.urdf.xacro (robot description, xacro)
@@ -13,5 +13,5 @@
       <visual>
         <geometry>
-          <mesh filename="package://rolling/urdf/mesh/20230808_frameless/battery_module.dae" scale="0.001 0.001 0.001"/>
+          <mesh filename="package://rolling/urdf/mesh/20230808_frameless/battery_module.dae" />
         </geometry>
       </visual>

File: robots/rolling/urdf/20230808_frameless/link1.urdf.xacro (robot description, xacro)
@@ -13,5 +13,5 @@
       <visual>
         <geometry>
-          <mesh filename="package://rolling/urdf/mesh/20230808_frameless/link1_base.dae" scale="0.001 0.001 0.001"/>
+          <mesh filename="package://rolling/urdf/mesh/20230808_frameless/link1_base.dae" />
         </geometry>
       </visual>
@@ -33,5 +33,5 @@
       <visual>
         <geometry>
-          <mesh filename="package://rolling/urdf/mesh/20230808_frameless/link1_gimbal.dae" scale="0.001 0.001 0.001"/>
+          <mesh filename="package://rolling/urdf/mesh/20230808_frameless/link1_gimbal.dae" />
         </geometry>
       </visual>

File: robots/rolling/urdf/20230808_frameless/link2.urdf.xacro (robot description, xacro)
@@ -13,5 +13,5 @@
       <visual>
         <geometry>
-          <mesh filename="package://rolling/urdf/mesh/20230808_frameless/link2_base.dae" scale="0.001 0.001 0.001"/>
+          <mesh filename="package://rolling/urdf/mesh/20230808_frameless/link2_base.dae" />
         </geometry>
       </visual>
@@ -33,5 +33,5 @@
       <visual>
         <geometry>
-          <mesh filename="package://rolling/urdf/mesh/20230808_frameless/link2_gimbal.dae" scale="0.001 0.001 0.001"/>
+          <mesh filename="package://rolling/urdf/mesh/20230808_frameless/link2_gimbal.dae" />
         </geometry>
       </visual>

File: robots/rolling/urdf/20230808_frameless/link3.urdf.xacro (robot description, xacro)
@@ -13,5 +13,5 @@
       <visual>
         <geometry>
-          <mesh filename="package://rolling/urdf/mesh/20230808_frameless/link3_base.dae" scale="0.001 0.001 0.001"/>
+          <mesh filename="package://rolling/urdf/mesh/20230808_frameless/link3_base.dae" />
         </geometry>
       </visual>
@@ -33,5 +33,5 @@
       <visual>
         <geometry>
-          <mesh filename="package://rolling/urdf/mesh/20230808_frameless/link3_gimbal.dae" scale="0.001 0.001 0.001"/>
+          <mesh filename="package://rolling/urdf/mesh/20230808_frameless/link3_gimbal.dae" />
         </geometry>
       </visual>

File: robots/rolling/urdf/shelled/rolling_link.urdf.xacro (robot description, xacro)
@@ -19,5 +19,5 @@
         <origin rpy="0 0 0" xyz="0 0 0"/>
         <geometry>
-          <mesh filename="package://rolling/urdf/mesh/shelled/link.dae" scale="0.001 0.001 0.001"/>
+          <mesh filename="package://rolling/urdf/mesh/shelled/link.dae" />
         </geometry>
         <xacro:glay/>
@@ -115,5 +115,5 @@
         </xacro:if>
         <geometry>
-          <mesh filename="package://rolling/urdf/mesh/shelled/roll_gimbal_module.dae" scale="0.001 0.001 0.001"/>
+          <mesh filename="package://rolling/urdf/mesh/shelled/roll_gimbal_module.dae" />
         </geometry>
         <xacro:black/>
