Commit message: [WIP] add external pipe to urdf for gain tuing

File: robots/rolling/urdf/20230808_frameless/link3.urdf.xacro (robot description, xacro)
@@ -37,4 +37,18 @@
       </visual>
     </link>
+    <link name="external_pipe">
+      <inertial>
+        <origin xyz="0 0 0" rpy="0 0 0"/>
+        <mass value="0.07"/>
+        <inertia
+            ixx="0.00001" iyy="0.00001" izz="0.00001"
+            ixy="0.00000" ixz="0.00000" iyz="0.00000"/>
+      </inertial>
+    </link>
+    <joint name="external_pipe_joint" type="fixed">
+      <parent link="link3"/>
+      <child link="external_pipe"/>
+      <origin xyz="0.75 0 0"/>
+    </joint>
   </xacro:macro>
 </robot>

Commit message: Revert "[WIP] add external pipe to urdf for gain tuing"
This reverts commit fd37320cbffb49db8640a325334fad599dd7b6d6.

File: robots/rolling/urdf/20230808_frameless/link3.urdf.xacro (robot description, xacro)
@@ -37,18 +37,4 @@
       </visual>
     </link>
-    <link name="external_pipe">
-      <inertial>
-        <origin xyz="0 0 0" rpy="0 0 0"/>
-        <mass value="0.07"/>
-        <inertia
-            ixx="0.00001" iyy="0.00001" izz="0.00001"
-            ixy="0.00000" ixz="0.00000" iyz="0.00000"/>
-      </inertial>
-    </link>
-    <joint name="external_pipe_joint" type="fixed">
-      <parent link="link3"/>
-      <child link="external_pipe"/>
-      <origin xyz="0.75 0 0"/>
-    </joint>
   </xacro:macro>
 </robot>
