Commit message: [rolling][urdf] replace meshed to armored version

File: robots/rolling/urdf/20231013_frame/link1.urdf.xacro (robot description, xacro)
@@ -13,5 +13,5 @@
       <visual>
         <geometry>
-          <mesh filename="package://rolling/urdf/mesh/20231013_frame/link1_base.dae" />
+          <mesh filename="package://rolling/urdf/mesh/20231013_frame/link1_base.stl" />
         </geometry>
       </visual>

File: robots/rolling/urdf/20231013_frame/link2.urdf.xacro (robot description, xacro)
@@ -13,5 +13,5 @@
       <visual>
         <geometry>
-          <mesh filename="package://rolling/urdf/mesh/20231013_frame/link2_base.dae" />
+          <mesh filename="package://rolling/urdf/mesh/20231013_frame/link2_base.stl" />
         </geometry>
       </visual>

File: robots/rolling/urdf/20231013_frame/link3.urdf.xacro (robot description, xacro)
@@ -13,5 +13,5 @@
       <visual>
         <geometry>
-          <mesh filename="package://rolling/urdf/mesh/20231013_frame/link3_base.dae" />
+          <mesh filename="package://rolling/urdf/mesh/20231013_frame/link3_base.stl" />
         </geometry>
       </visual>

Commit message: [rolling][urdf] update inertial parameter of armored type

File: robots/rolling/urdf/20231013_frame/link1.urdf.xacro (robot description, xacro)
@@ -5,9 +5,9 @@
     <link name="link1">
       <inertial>
-        <origin xyz="0.26695257 0.00000500 0.00993736" rpy="0 0 0"/>
-        <mass value="0.48484449"/>
+        <origin xyz="0.26901888 -0.03575861 0.00778837" rpy="0 0 0"/>
+        <mass value="0.70811094"/>
         <inertia
-            ixx="0.00050326"  iyy="0.01670962" izz="0.01633157"
-            ixy="-0.00000023" ixz="0.00133774" iyz="0.00000004"/>
+            ixx="0.00344639"  iyy="0.02416547" izz="0.02611708"
+            ixy="0.00055924"  ixz="0.00141558" iyz="0.00019727"/>
       </inertial>
       <visual>

File: robots/rolling/urdf/20231013_frame/link2.urdf.xacro (robot description, xacro)
@@ -5,9 +5,9 @@
     <link name="link2">
       <inertial>
-        <origin xyz="0.26724120 -0.00000341 0.00917818" rpy="0 0 0"/>
-        <mass value="0.55395179"/>
+        <origin xyz="0.27923148 -0.03253302 0.00743660" rpy="0 0 0"/>
+        <mass value="0.77749010"/>
         <inertia
-            ixx="0.00055160"  iyy="0.02080064" izz="0.02042362"
-            ixy="-0.00000055" ixz="0.00153902" iyz="-0.00000007"/>
+            ixx="0.00357609"  iyy="0.02868885" izz="0.03072531"
+            ixy="-0.00002501" ixz="0.00160483" iyz="-0.00018947"/>
       </inertial>
       <visual>

File: robots/rolling/urdf/20231013_frame/link3.urdf.xacro (robot description, xacro)
@@ -5,9 +5,9 @@
     <link name="link3">
       <inertial>
-        <origin xyz="0.21323824 0.00000000 -0.00885891" rpy="0 0 0"/>
-        <mass value="0.34751322"/>
+        <origin xyz="0.24636697 -0.04526078 -0.00550471" rpy="0 0 0"/>
+        <mass value="0.55950172"/>
         <inertia
-            ixx="0.00041721" iyy="0.01179645"  izz="0.01149579"
-            ixy="0.00000000" ixz="-0.00026812" iyz="0.00000000"/>
+            ixx="0.00308740"  iyy="0.02009202"  izz="0.02191011"
+            ixy="-0.00086249" ixz="-0.00016618" iyz="-0.00013940"/>
       </inertial>
       <visual>

Commit message: [rolling] replace stl to dae

File: robots/rolling/urdf/20231013_frame/link1.urdf.xacro (robot description, xacro)
@@ -13,5 +13,5 @@
       <visual>
         <geometry>
-          <mesh filename="package://rolling/urdf/mesh/20231013_frame/link1_base.stl" />
+          <mesh filename="package://rolling/urdf/mesh/20231013_frame/link1_base.dae" />
         </geometry>
       </visual>

File: robots/rolling/urdf/20231013_frame/link2.urdf.xacro (robot description, xacro)
@@ -13,5 +13,5 @@
       <visual>
         <geometry>
-          <mesh filename="package://rolling/urdf/mesh/20231013_frame/link2_base.stl" />
+          <mesh filename="package://rolling/urdf/mesh/20231013_frame/link2_base.dae" />
         </geometry>
       </visual>

File: robots/rolling/urdf/20231013_frame/link3.urdf.xacro (robot description, xacro)
@@ -13,5 +13,5 @@
       <visual>
         <geometry>
-          <mesh filename="package://rolling/urdf/mesh/20231013_frame/link3_base.stl" />
+          <mesh filename="package://rolling/urdf/mesh/20231013_frame/link3_base.dae" />
         </geometry>
       </visual>
