Commit message: [rolling] update urdf

File: robots/rolling/urdf/20231013_frame/rolling_link.urdf.xacro (robot description, xacro)
@@ -117,5 +117,5 @@
         <collision>
           <geometry>
-            <cylinder radius="0.4" length="0.1"/>
+            <cylinder radius="0.405" length="0.1"/>
           </geometry>
         </collision>

File: robots/rolling/urdf/common.xacro (robot description, xacro)
@@ -18,6 +18,6 @@
   <xacro:macro name="large_friction" params="link">
     <gazebo reference="${link}">
-      <mu1>20</mu1>
-      <mu2>20</mu2>
+      <mu1>100</mu1>
+      <mu2>100</mu2>
     </gazebo>
   </xacro:macro>

Commit message: [rolling][urdf] update thickness of cylinder for collision

File: robots/rolling/urdf/20231013_frame/rolling_link.urdf.xacro (robot description, xacro)
@@ -117,5 +117,5 @@
         <collision>
           <geometry>
-            <cylinder radius="0.405" length="0.1"/>
+            <cylinder radius="0.405" length="0.03"/>
           </geometry>
         </collision>

Commit message: [rolling][urdf] remove upper and lower limit for gimbal joint

File: robots/rolling/urdf/20231013_frame/rolling_link.urdf.xacro (robot description, xacro)
@@ -56,5 +56,5 @@
     <!-- gimbal joint -->
     <joint name="gimbal${self}" type="continuous">
-      <limit effort="3" lower="-3.14" upper="3.14" velocity="12.5"/>
+      <limit effort="3" velocity="12.5"/>
       <parent link="link${self}"/>
       <child link="gimbal_link${self}"/>

Commit message: Revert "[rolling][urdf] remove upper and lower limit for gimbal joint"
This reverts commit cce6d97daeb03ec0a450f899eaa5bd4dd7db192e.

File: robots/rolling/urdf/20231013_frame/rolling_link.urdf.xacro (robot description, xacro)
@@ -56,5 +56,5 @@
     <!-- gimbal joint -->
     <joint name="gimbal${self}" type="continuous">
-      <limit effort="3" velocity="12.5"/>
+      <limit effort="3" lower="-3.14" upper="3.14" velocity="12.5"/>
       <parent link="link${self}"/>
       <child link="gimbal_link${self}"/>

Commit message: [rolling][control] solve the round offset problem in gimbal control

File: robots/rolling/urdf/20231013_frame/rolling_link.urdf.xacro (robot description, xacro)
@@ -56,5 +56,5 @@
     <!-- gimbal joint -->
     <joint name="gimbal${self}" type="continuous">
-      <limit effort="3" lower="-3.14" upper="3.14" velocity="12.5"/>
+      <limit effort="3" lower="-15.0" upper="15.0" velocity="12.5"/>
       <parent link="link${self}"/>
       <child link="gimbal_link${self}"/>
