Commit message: [delta][control] workaround nonlinear wrench allocation with pinocchio and casadi

File: robots/delta/urdf/20240207_new_armor/rolling_link.urdf.xacro (robot description, xacro)
@@ -55,5 +55,5 @@
     </xacro:if>
     <!-- gimbal joint -->
-    <joint name="gimbal${self}" type="continuous">
+    <joint name="gimbal${self}" type="revolute">
       <limit effort="3" lower="-15.0" upper="15.0" velocity="12.5"/>
       <parent link="link${self}"/>
