Commit message: [delta] add new robot type 20240319_mesh. its collision model is based on optimized mesh

File: robots/delta/urdf/common.xacro (robot description, xacro)
@@ -19,4 +19,6 @@
     </gazebo>
   </xacro:macro>
+  <!-- leg length -->
+  <xacro:property name="leg_length" value="0.135"/>
   <xacro:macro name="damping_factor" params="link">
     <gazebo reference="${link}">
