Commit message: [delta][urdf] refactor urdf

File: robots/delta/urdf/20240319_mesh/link1.urdf.xacro (robot description, xacro)
@@ -5,12 +5,5 @@
     <!-- dummy root link for KDL -->
     <link name="root">
-      <inertial>
-        <origin xyz="0 0 0" rpy="0 0 0"/>
-        <mass value="0.00001"/>
-        <inertia
-            ixx="0.000001" ixy="0.0" ixz="0.0"
-            iyy="0.000001" iyz="0.0"
-            izz="0.000001"/>
-      </inertial>
+      <xacro:virtual_inertial/>
     </link>
     <joint name="root_joint" type="fixed">
@@ -43,13 +36,13 @@
     <link name="link1_leg">
       <inertial>
-        <mass value="0.00001"/>
+        <mass value="${leg_mass}"/>
         <inertia
-            ixx="0.000001" ixy="0.0" ixz="0.0"
-            iyy="0.000001" iyz="0.0"
-            izz="0.000001"/>
+            ixx="${(leg_radius * leg_radius / 4.0 + leg_length * leg_length / 12.0) * leg_mass}" ixy="0.0" ixz="0.0"
+            iyy="${(leg_radius * leg_radius / 4.0 + leg_length * leg_length / 12.0) * leg_mass}" iyz="0.0"
+            izz="${(leg_radius * leg_radius / 2.0) * leg_mass}"/>
       </inertial>
       <collision>
         <geometry>
-          <cylinder radius="0.012" length="${leg_length}"/>
+          <cylinder radius="${leg_radius}" length="${leg_length}"/>
         </geometry>
       </collision>
@@ -76,12 +69,5 @@
     </link>
     <link name="link1_center">
-      <inerial>
-        <origin xyz="0 0 0"/>
-          <mass value="0.00001"/>
-          <inertia
-              ixx="0.000004" ixy="0.0" ixz="0.0"
-              iyy="0.000004" iyz="0.0"
-              izz="0.000004"/>
-      </inerial>
+      <xacro:virtual_inertial/>
     </link>
     <joint name="link1_center_joint" type="fixed">

File: robots/delta/urdf/20240319_mesh/link2.urdf.xacro (robot description, xacro)
@@ -5,12 +5,5 @@
     <!-- fc frame -->
     <link name="fc">
-      <inertial>
-        <origin xyz="0 0 0" rpy="0 0 0"/>
-        <mass value="0.00001"/>
-        <inertia
-            ixx="0.000001" ixy="0.0" ixz="0.0"
-            iyy="0.000001" iyz="0.0"
-            izz="0.000002"/>
-      </inertial>
+      <xacro:virtual_inertial/>
     </link>
     <joint name="fc_joint" type="fixed">
@@ -43,13 +36,13 @@
     <link name="link2_leg">
       <inertial>
-        <mass value="0.00001"/>
+        <mass value="${leg_mass}"/>
         <inertia
-            ixx="0.000001" ixy="0.0" ixz="0.0"
-            iyy="0.000001" iyz="0.0"
-            izz="0.000001"/>
+            ixx="${(leg_radius * leg_radius / 4.0 + leg_length * leg_length / 12.0) * leg_mass}" ixy="0.0" ixz="0.0"
+            iyy="${(leg_radius * leg_radius / 4.0 + leg_length * leg_length / 12.0) * leg_mass}" iyz="0.0"
+            izz="${(leg_radius * leg_radius / 2.0) * leg_mass}"/>
       </inertial>
       <collision>
         <geometry>
-          <cylinder radius="0.012" length="${leg_length}"/>
+          <cylinder radius="${leg_radius}" length="${leg_length}"/>
         </geometry>
       </collision>
@@ -76,12 +69,5 @@
     </link>
     <link name="link2_center">
-      <inerial>
-        <origin xyz="0 0 0"/>
-          <mass value="0.00001"/>
-          <inertia
-              ixx="0.000001" ixy="0.0" ixz="0.0"
-              iyy="0.000001" iyz="0.0"
-              izz="0.000001"/>
-      </inerial>
+      <xacro:virtual_inertial/>
     </link>
     <joint name="link2_center_joint" type="fixed">

File: robots/delta/urdf/20240319_mesh/link3.urdf.xacro (robot description, xacro)
@@ -26,13 +26,13 @@
     <link name="link3_leg1">
       <inertial>
-        <mass value="0.00001"/>
+        <mass value="${leg_mass}"/>
         <inertia
-            ixx="0.000001" ixy="0.0" ixz="0.0"
-            iyy="0.000001" iyz="0.0"
-            izz="0.000001"/>
+            ixx="${(leg_radius * leg_radius / 4.0 + leg_length * leg_length / 12.0) * leg_mass}" ixy="0.0" ixz="0.0"
+            iyy="${(leg_radius * leg_radius / 4.0 + leg_length * leg_length / 12.0) * leg_mass}" iyz="0.0"
+            izz="${(leg_radius * leg_radius / 2.0) * leg_mass}"/>
       </inertial>
       <collision>
         <geometry>
-          <cylinder radius="0.012" length="${leg_length}"/>
+          <cylinder radius="${leg_radius}" length="${leg_length}"/>
         </geometry>
       </collision>
@@ -46,9 +46,9 @@
     <link name="link3_leg2">
       <inertial>
-        <mass value="0.00001"/>
+        <mass value="${leg_mass}"/>
         <inertia
-            ixx="0.000001" ixy="0.0" ixz="0.0"
-            iyy="0.000001" iyz="0.0"
-            izz="0.000001"/>
+            ixx="${(leg_radius * leg_radius / 4.0 + leg_length * leg_length / 12.0) * leg_mass}" ixy="0.0" ixz="0.0"
+            iyy="${(leg_radius * leg_radius / 4.0 + leg_length * leg_length / 12.0) * leg_mass}" iyz="0.0"
+            izz="${(leg_radius * leg_radius / 2.0) * leg_mass}"/>
       </inertial>
       <collision>
@@ -79,12 +79,5 @@
     </link>
     <link name="link3_center">
-      <inerial>
-        <origin xyz="0 0 0"/>
-          <mass value="0.00001"/>
-          <inertia
-              ixx="0.000001" ixy="0.0" ixz="0.0"
-              iyy="0.000001" iyz="0.0"
-              izz="0.000001"/>
-      </inerial>
+      <xacro:virtual_inertial/>
     </link>
     <joint name="link3_center_joint" type="fixed">

File: robots/delta/urdf/20240319_mesh/rolling_link.urdf.xacro (robot description, xacro)
@@ -57,5 +57,5 @@
             ixx="0.000001" ixy="0.0" ixz="0.0"
             iyy="0.000001" iyz="0.0"
-            izz="0.000001"/>
+            izz="0.000002"/>
       </inertial>
     </link>
@@ -82,5 +82,5 @@
             ixx="0.000001" ixy="0.0" ixz="0.0"
             iyy="0.000001" iyz="0.0"
-            izz="0.000001"/>
+            izz="0.000002"/>
       </inertial>
     </link>

File: robots/delta/urdf/common.xacro (robot description, xacro)
@@ -19,6 +19,19 @@
     </gazebo>
   </xacro:macro>
-  <!-- leg length -->
+  <!-- leg -->
   <xacro:property name="leg_length" value="0.135"/>
+  <xacro:property name="leg_mass" value="0.01"/>
+  <xacro:property name="leg_radius" value="0.006"/>
+  <!-- macro of inertial of virtual link -->
+  <xacro:macro name="virtual_inertial" params="x:=0 y:=0 z:=0">
+    <inerial>
+      <origin xyz="${x} ${y} ${z}"/>
+      <mass value="0.00001"/>
+      <inertia
+          ixx="0.000001" ixy="0.0" ixz="0.0"
+          iyy="0.000001" iyz="0.0"
+          izz="0.000002"/>
+    </inerial>
+  </xacro:macro>
   <xacro:macro name="damping_factor" params="link">
     <gazebo reference="${link}">
@@ -26,13 +39,3 @@
     </gazebo>
   </xacro:macro>
-  <xacro:macro name="glay">
-    <material name="glay" >
-      <color rgba="0.5 0.5 0.5 1.0" />
-    </material>
-  </xacro:macro>
-  <xacro:macro name="black">
-    <material name="black" >
-      <color rgba="0 0 0 1.0" />
-    </material>
-  </xacro:macro>
 </robot>
