Commit message: [delta] add link3_end frame in urdf

File: robots/delta/urdf/20240319_mesh/link3.urdf.xacro (robot description, xacro)
@@ -23,4 +23,12 @@
     </link>
     <xacro:large_friction link="link3"/>
+    <link name="link3_end">
+      <xacro:virtual_inertial/>
+    </link>
+    <joint name="link3_end_joint" type="fixed">
+      <parent link="link3"/>
+      <child link="link3_end"/>
+      <origin xyz="0.5335 0  0" rpy="0 0 0"/>
+    </joint>
     <!-- leg -->
     <link name="link3_leg1">
