Commit message: [delta] update door opening demo

File: robots/delta/urdf/demo/door.urdf (robot description, URDF)
Before this commit: robot door, 3 links, 2 joints
Links:
- removed link door_base
- added link base_link, mass 10.0; collision box size=1 1 2; visual box size=1 1 2
- link door_knob_link: geometry collision cylinder length=${door_knob_length} radius=0.02; visual cylinder length=${door_knob_length} radius=0.02
Joints:
- joint door_knob_joint: origin xyz=-0.2 0.5 0 -> xyz=-0.2 -0.5 0
- joint slide_door_joint: origin xyz=-0.5 0 1 -> xyz=-0.5 0.5 1; parent door_base -> base_link
