Commit message: [delta] add new robot type

File: robots/delta/urdf/20240722/link1.urdf.xacro (robot description, xacro)
@@ -15,9 +15,9 @@
     <link name="link1">
       <inertial>
-        <origin xyz="0.28794398 -0.04712329 0.00347969" rpy="0 0 0"/>
-        <mass value="1.08222549"/>
+        <origin xyz="0.27442477 -0.04145571 0.00766623" rpy="0 0 0"/>
+        <mass value="0.80165566"/>
         <inertia
-             ixx="0.00498184" iyy="0.03252549" izz="0.03516989"
-            ixy="-0.00088064" ixz="0.00165575" iyz="0.00017753" />
+             ixx="0.00393460" iyy="0.02769902" izz="0.03031993"
+            ixy="-0.00001765" ixz="0.00072820" iyz="0.00025451" />
       </inertial>
       <visual>
@@ -56,9 +56,9 @@
     <link name="gimbal_link1">
       <inertial>
-        <origin xyz="0.00944096 -0.00000223 0.01141561" rpy="0 0 0"/>
-        <mass value="0.27443334"/>
+        <origin xyz="0.00787449 -0.00000198 0.01067283" rpy="0 0 0"/>
+        <mass value="0.30953004"/>
         <inertia
-            ixx="0.00066652"  iyy="0.00074131" izz="0.00017798"
-            ixy="0.00000004" ixz="-0.00017867" iyz="0.00000005" />
+            ixx="0.00077572"  iyy="0.00085410" izz="0.00019463"
+            ixy="0.00000000" ixz="-0.00017623" iyz="0.00000005" />
       </inertial>
       <visual>

File: robots/delta/urdf/20240722/link2.urdf.xacro (robot description, xacro)
@@ -15,9 +15,9 @@
     <link name="link2">
       <inertial>
-        <origin xyz="0.29247546 -0.04173228 0.00214003" rpy="0 0 0"/>
-        <mass value="1.21919627"/>
+        <origin xyz="0.27430376 -0.03531382 0.00536770" rpy="0 0 0"/>
+        <mass value="0.93865101"/>
         <inertia
-             ixx="0.00538607" iyy="0.04105715" izz="0.04397541"
-            ixy="-0.00237976" ixz="0.00218016" iyz="0.00011267" />
+             ixx="0.00427555" iyy="0.03420212" izz="0.03701377"
+            ixy="-0.00115915" ixz="0.00112391" iyz="0.00018003" />
       </inertial>
       <visual>
@@ -56,9 +56,9 @@
     <link name="gimbal_link2">
       <inertial>
-        <origin xyz="0.01205240 -0.00000221 0.01260343" rpy="0 0 0"/>
-        <mass value="0.27751558"/>
+        <origin xyz="0.01035776 -0.00000204 0.01055007" rpy="0 0 0"/>
+        <mass value="0.30812645"/>
         <inertia
-            ixx="0.00068946"  iyy="0.00075023" izz="0.00016497"
-            ixy="0.00000004" ixz="-0.00015101" iyz="0.00000005"/>
+            ixx="0.00077363"  iyy="0.00083923" izz="0.00018147"
+            ixy="0.00000000" ixz="-0.00014207" iyz="0.00000005"/>
       </inertial>
       <visual>

File: robots/delta/urdf/20240722/link3.urdf.xacro (robot description, xacro)
@@ -5,9 +5,9 @@
     <link name="link3">
       <inertial>
-        <origin xyz="0.29164273 -0.05294374 -0.00632002" rpy="0 0 0"/>
-        <mass value="0.95975816"/>
+        <origin xyz="0.26112729 -0.04939508 0.00100978" rpy="0 0 0"/>
+        <mass value="0.66898892"/>
         <inertia
-             ixx="0.00478040"  iyy="0.03231099"  izz="0.03458590"
-            ixy="-0.00244503"  ixz="0.00009334" iyz="-0.00032114" />
+             ixx="0.00346166"  iyy="0.02400775"  izz="0.02657264"
+            ixy="-0.00160932" ixz="-0.00014653"  iyz="0.00003337" />
       </inertial>
       <visual>
@@ -74,9 +74,9 @@
     <link name="gimbal_link3">
       <inertial>
-        <origin xyz="0.00935372 -0.00000228 0.01150070" rpy="0 0 0"/>
-        <mass value="0.27464497"/>
+        <origin xyz="0.00779810 -0.00000202 0.01075117" rpy="0 0 0"/>
+        <mass value="0.30974142"/>
         <inertia
-            ixx="0.00066816"  iyy="0.00074345"  izz="0.00017856"
-            ixy="0.00000004" ixz="-0.00017982"  iyz="0.00000005" />
+            ixx="0.00077756"  iyy="0.00085638"  izz="0.00019513"
+            ixy="0.00000000" ixz="-0.00017744"  iyz="0.00000005" />
       </inertial>
       <visual>

File: robots/delta/urdf/20240722/rolling_link.urdf.xacro (robot description, xacro)
@@ -2,9 +2,10 @@
 <robot
     xmlns:xacro="http://www.ros.org/wiki/xacro" name="delta_link" >
-  <xacro:include filename="$(find delta)/urdf/20240319_mesh/link1.urdf.xacro" />
-  <xacro:include filename="$(find delta)/urdf/20240319_mesh/link2.urdf.xacro" />
-  <xacro:include filename="$(find delta)/urdf/20240319_mesh/link3.urdf.xacro" />
-  <xacro:include filename="$(find delta)/urdf/20240319_mesh/thrust.urdf.xacro" />
-  <xacro:macro name="delta_module" params="self child rotor_direction">
+  <xacro:include filename="$(find delta)/urdf/20240722/link1.urdf.xacro" />
+  <xacro:include filename="$(find delta)/urdf/20240722/link2.urdf.xacro" />
+  <xacro:include filename="$(find delta)/urdf/20240722/link3.urdf.xacro" />
+  <xacro:include filename="$(find delta)/urdf/20240722/thrust.urdf.xacro" />
+  <xacro:include filename="$(find delta)/urdf/20240722/battery.urdf.xacro" />
+  <xacro:macro name="delta_module" params="self child rotor_direction battery">
     <xacro:if value="${self == 1}">
       <xacro:link1/>
@@ -93,4 +94,21 @@
       <axis xyz="0 0 ${rotor_direction}"/>
     </joint>
+    <!-- battery -->
+    <xacro:if value="${battery == 1}">
+      <xacro:high_lipo_single index="${self}"/>
+      <joint name="battery_joint${self}" type="fixed">
+        <parent link="link${self}"/>
+        <child link="high_lipo_single${self}"/>
+        <xacro:if value="${self == 1}">
+          <origin xyz="0.3735 -0.038 0" rpy="${pi / 2} 0 ${-pi / 2}"/>
+        </xacro:if>
+        <xacro:if value="${self == 2}">
+          <origin xyz="0.407 -0.038 0" rpy="${pi / 2} 0 ${-pi / 2}"/>
+        </xacro:if>
+        <xacro:if value="${self == 3}">
+          <origin xyz="0.407 -0.038 0" rpy="${pi / 2} 0 ${-pi / 2}"/>
+        </xacro:if>
+      </joint>
+    </xacro:if>
     <!-- hardware interface -->
     <xacro:unless value="${self == child}">
