Commit message: [delta] update urdf model

File: robots/delta/urdf/20240722/battery.urdf.xacro (robot description, xacro)
@@ -14,5 +14,5 @@
       <visual>
         <geometry>
-          <mesh filename="package://delta/urdf/mesh/20240117_10inch/high_lipo_single_module.stl" />
+          <mesh filename="package://delta/urdf/mesh/20240722/high_lipo_single_module.stl" />
         </geometry>
       </visual>

File: robots/delta/urdf/20240722/link1.urdf.xacro (robot description, xacro)
@@ -23,10 +23,10 @@
       <visual>
         <geometry>
-          <mesh filename="package://delta/urdf/mesh/20240319_mesh/link1_base.dae" />
+          <mesh filename="package://delta/urdf/mesh/20240722/link1_base.dae" />
         </geometry>
       </visual>
       <collision>
         <geometry>
-          <mesh filename="package://delta/urdf/mesh/20240319_mesh/link1_base_opt.stl" />
+          <mesh filename="package://delta/urdf/mesh/20240722/link1_base_opt.stl" />
         </geometry>
       </collision>
@@ -64,5 +64,5 @@
       <visual>
         <geometry>
-          <mesh filename="package://delta/urdf/mesh/20240319_mesh/link1_gimbal.dae" />
+          <mesh filename="package://delta/urdf/mesh/20240722/link1_gimbal.dae" />
         </geometry>
       </visual>

File: robots/delta/urdf/20240722/link2.urdf.xacro (robot description, xacro)
@@ -23,10 +23,10 @@
       <visual>
         <geometry>
-          <mesh filename="package://delta/urdf/mesh/20240319_mesh/link2_base.dae" />
+          <mesh filename="package://delta/urdf/mesh/20240722/link2_base.dae" />
         </geometry>
       </visual>
       <collision>
         <geometry>
-          <mesh filename="package://delta/urdf/mesh/20240319_mesh/link2_base_opt.stl" />
+          <mesh filename="package://delta/urdf/mesh/20240722/link2_base_opt.stl" />
         </geometry>
       </collision>
@@ -64,5 +64,5 @@
       <visual>
         <geometry>
-          <mesh filename="package://delta/urdf/mesh/20240319_mesh/link2_gimbal.dae" />
+          <mesh filename="package://delta/urdf/mesh/20240722/link2_gimbal.dae" />
         </geometry>
       </visual>

File: robots/delta/urdf/20240722/link3.urdf.xacro (robot description, xacro)
@@ -13,10 +13,10 @@
       <visual>
         <geometry>
-          <mesh filename="package://delta/urdf/mesh/20240319_mesh/link3_base.dae" />
+          <mesh filename="package://delta/urdf/mesh/20240722/link3_base.dae" />
         </geometry>
       </visual>
       <collision>
         <geometry>
-          <mesh filename="package://delta/urdf/mesh/20240319_mesh/link3_base_opt.stl" />
+          <mesh filename="package://delta/urdf/mesh/20240722/link3_base_opt.stl" />
         </geometry>
       </collision>
@@ -82,5 +82,5 @@
       <visual>
         <geometry>
-          <mesh filename="package://delta/urdf/mesh/20240319_mesh/link3_gimbal.dae" />
+          <mesh filename="package://delta/urdf/mesh/20240722/link3_gimbal.dae" />
         </geometry>
       </visual>
