Commit message: [delta][control] refactor nonlinear optimization and add constraint function about joint torque

File: robots/delta/urdf/20240722/rolling_link.urdf.xacro (robot description, xacro)
@@ -24,4 +24,37 @@
       <axis xyz="1 0 0"/>
       <dynamics damping="0.1" friction="0.0"/>
+      <xacro:if value="${self == 1}">
+        <origin xyz="0.170 0 0" rpy="0 0 0" />
+      </xacro:if>
+      <xacro:if value="${self == 2}">
+        <origin xyz="0.2035 0 0" rpy="0 0 0" />
+      </xacro:if>
+      <xacro:if value="${self == 3}">
+        <origin xyz="0.2035 0 0" rpy="0 0 0" />
+      </xacro:if>
+    </joint>
+    <!-- gimbal neutral coord -->
+    <link name="gimbal_neutral_coord${self}">
+      <inertial>
+        <xacro:if value="${self == 1}">
+          <origin xyz="0 0 0" rpy="0 0 0" />
+        </xacro:if>
+        <xacro:if value="${self == 2}">
+          <origin xyz="0 0 0" rpy="0 0 0" />
+        </xacro:if>
+        <xacro:if value="${self == 3}">
+          <origin xyz="0 0 0" rpy="0 0 0" />
+        </xacro:if>
+        <mass value="0.00001"/>
+        <inertia
+            ixx="0.000001" ixy="0.0" ixz="0.0"
+            iyy="0.000001" iyz="0.0"
+            izz="0.000002"/>
+      </inertial>
+    </link>
+    <joint name="gimbal_neutral_coord_joint${self}" type="fixed">
+      <parent link="link${self}"/>
+      <child link="gimbal_neutral_coord${self}"/>
+      <axis xyz="0 0 1"/>
       <xacro:if value="${self == 1}">
         <origin xyz="0.170 0 0" rpy="0 0 0" />

Commit message: [delta][urdf] update joint parameter corresponding to real machine

File: robots/delta/urdf/20240722/rolling_link.urdf.xacro (robot description, xacro)
@@ -70,5 +70,5 @@
     <xacro:unless value="${self == child}">
       <joint name="joint${self}" type="revolute" >
-        <limit effort="20.0" lower="${-pi}" upper="${pi}" velocity="0.1"/>
+        <limit effort="6.8" lower="${-pi}" upper="${pi * 2 / 3}" velocity="0.1755"/>
         <parent link="link${self}" />
         <child  link="link${child}" />

Commit message: [delta][control] removed gimbal neutral coordinate and changed frame used for gimbal jacobian

File: robots/delta/urdf/20240722/rolling_link.urdf.xacro (robot description, xacro)
@@ -24,37 +24,4 @@
       <axis xyz="1 0 0"/>
       <dynamics damping="0.1" friction="0.0"/>
-      <xacro:if value="${self == 1}">
-        <origin xyz="0.170 0 0" rpy="0 0 0" />
-      </xacro:if>
-      <xacro:if value="${self == 2}">
-        <origin xyz="0.2035 0 0" rpy="0 0 0" />
-      </xacro:if>
-      <xacro:if value="${self == 3}">
-        <origin xyz="0.2035 0 0" rpy="0 0 0" />
-      </xacro:if>
-    </joint>
-    <!-- gimbal neutral coord -->
-    <link name="gimbal_neutral_coord${self}">
-      <inertial>
-        <xacro:if value="${self == 1}">
-          <origin xyz="0 0 0" rpy="0 0 0" />
-        </xacro:if>
-        <xacro:if value="${self == 2}">
-          <origin xyz="0 0 0" rpy="0 0 0" />
-        </xacro:if>
-        <xacro:if value="${self == 3}">
-          <origin xyz="0 0 0" rpy="0 0 0" />
-        </xacro:if>
-        <mass value="0.00001"/>
-        <inertia
-            ixx="0.000001" ixy="0.0" ixz="0.0"
-            iyy="0.000001" iyz="0.0"
-            izz="0.000002"/>
-      </inertial>
-    </link>
-    <joint name="gimbal_neutral_coord_joint${self}" type="fixed">
-      <parent link="link${self}"/>
-      <child link="gimbal_neutral_coord${self}"/>
-      <axis xyz="0 0 1"/>
       <xacro:if value="${self == 1}">
         <origin xyz="0.170 0 0" rpy="0 0 0" />
