Commit message: [delta] refactor urdf: separate fc and link2. link number can be changed

File: robots/delta/robots/20240722/rolling.urdf.xacro (robot description, xacro)
@@ -4,6 +4,6 @@
   <xacro:include filename="$(find delta)/urdf/20240722/rolling_link.urdf.xacro" />
   <xacro:include filename="$(find delta)/urdf/common.xacro" />
-  <xacro:delta_module self="1" child="2" rotor_direction="1" battery="0"/>
-  <xacro:delta_module self="2" child="3" rotor_direction="-1" battery="0"/>
-  <xacro:delta_module self="3" child="3" rotor_direction="1" battery="0"/>
+  <xacro:delta_module self="1" child="2" rotor_direction="1" battery="0" baselink="false"/>
+  <xacro:delta_module self="2" child="3" rotor_direction="-1" battery="0" baselink="true"/>
+  <xacro:delta_module self="3" child="3" rotor_direction="1" battery="0" baselink="false"/>
 </robot>

File: robots/delta/urdf/20240722/link1.urdf.xacro (robot description, xacro)
@@ -3,14 +3,5 @@
     xmlns:xacro="http://www.ros.org/wiki/xacro" name="delta_link1" >
   <xacro:macro name="link1">
-    <!-- dummy root link for KDL -->
-    <link name="root">
-      <xacro:virtual_inertial/>
-    </link>
-    <joint name="root_joint" type="fixed">
-      <parent link="root"/>
-      <child link="link1"/>
-      <origin rpy="0 0 0" xyz="0 0 0"/>
-      <axis xyz="0 0 1"/>
-    </joint>
+    <!-- link -->
     <link name="link1">
       <inertial>
@@ -54,4 +45,5 @@
       <axis xyz="0 0 1"/>
     </joint>
+    <!-- gimbal -->
     <link name="gimbal_link1">
       <inertial>
@@ -68,4 +60,5 @@
       </visual>
     </link>
+    <!-- center of link -->
     <link name="link1_center">
       <xacro:virtual_inertial/>

File: robots/delta/urdf/20240722/link2.urdf.xacro (robot description, xacro)
@@ -3,21 +3,12 @@
     xmlns:xacro="http://www.ros.org/wiki/xacro" name="delta_link2" >
   <xacro:macro name="link2">
-    <!-- fc frame -->
-    <link name="fc">
-      <xacro:virtual_inertial/>
-    </link>
-    <joint name="fc_joint" type="fixed">
-      <child link="fc" />
-      <parent link="link2" />
-      <origin xyz="0.0864 -0.0012 0.020" rpy="0 0 0" />
-      <axis xyz="0 0 1"/>
-    </joint>
+    <!-- link -->
     <link name="link2">
       <inertial>
-        <origin xyz="0.27430376 -0.03531382 0.00536770" rpy="0 0 0"/>
-        <mass value="0.93865101"/>
+        <origin xyz="0.29984170 -0.04053992 0.00751982" rpy="0 0 0"/>
+        <mass value="0.81525662"/>
         <inertia
-             ixx="0.00427555" iyy="0.03420212" izz="0.03701377"
-            ixy="-0.00115915" ixz="0.00112391" iyz="0.00018003" />
+             ixx="0.00398803" iyy="0.02991643" izz="0.03256914"
+            ixy="-0.00033115" ixz="0.00077590" iyz="0.00024828" />
       </inertial>
       <visual>
@@ -54,4 +45,5 @@
       <axis xyz="0 0 1"/>
     </joint>
+    <!-- gimbal -->
     <link name="gimbal_link2">
       <inertial>
@@ -68,4 +60,5 @@
       </visual>
     </link>
+    <!-- center of link -->
     <link name="link2_center">
       <xacro:virtual_inertial/>

File: robots/delta/urdf/20240722/link3.urdf.xacro (robot description, xacro)
@@ -3,4 +3,5 @@
     xmlns:xacro="http://www.ros.org/wiki/xacro" name="delta_link3" >
   <xacro:macro name="link3">
+    <!-- link -->
     <link name="link3">
       <inertial>
@@ -23,4 +24,5 @@
     </link>
     <xacro:large_friction link="link3"/>
+    <!-- link end frame -->
     <link name="link3_end">
       <xacro:virtual_inertial/>
@@ -72,4 +74,5 @@
       <axis xyz="0 0 1"/>
     </joint>
+    <!-- gimbal -->
     <link name="gimbal_link3">
       <inertial>
@@ -86,4 +89,5 @@
       </visual>
     </link>
+    <!-- center of link -->
     <link name="link3_center">
       <xacro:virtual_inertial/>

File: robots/delta/urdf/20240722/rolling_link.urdf.xacro (robot description, xacro)
@@ -7,13 +7,53 @@
   <xacro:include filename="$(find delta)/urdf/20240722/thrust.urdf.xacro" />
   <xacro:include filename="$(find delta)/urdf/20240722/battery.urdf.xacro" />
-  <xacro:macro name="delta_module" params="self child rotor_direction battery">
+  <xacro:macro name="delta_module" params="self child rotor_direction battery baselink">
     <xacro:if value="${self == 1}">
       <xacro:link1/>
     </xacro:if>
-    <xacro:if value="${self == 2}">
+    <xacro:if value="${self != 1 and self != child}">
       <xacro:link2/>
     </xacro:if>
-    <xacro:if value="${self == 3}">
+    <xacro:if value="${self == child}">
       <xacro:link3/>
+    </xacro:if>
+    <!-- dummy root link for KDL -->
+    <xacro:if value="${self == 1}">
+      <link name="root">
+        <xacro:virtual_inertial/>
+      </link>
+      <joint name="root_joint" type="fixed">
+        <parent link="root"/>
+        <child link="link${self}"/>
+        <origin rpy="0 0 0" xyz="0 0 0"/>
+        <axis xyz="0 0 1"/>
+      </joint>
+    </xacro:if>
+    <!-- processors -->
+    <xacro:if value="${baselink}">
+      <link name="fc_link">
+        <xacro:virtual_inertial/>
+      </link>
+      <joint name="fc_link_joint" type="fixed">
+        <parent link="link${self}"/>
+        <child link="fc_link"/>
+        <axis xyz="0 0 1"/>
+        <origin xyz="0.0735 0 0" rpy="0 0 0"/>
+      </joint>
+      <link name="fc">
+        <inertial>
+          <origin xyz="0.02959036 -0.00076922 -0.00886856" rpy="0 0 0"/>
+          <mass value="0.12308403"/>
+          <inertia
+              ixx="0.00008649" ixy="-0.00000081" ixz="0.00000124"
+              iyy="0.00006899" iyz="0.00000148"
+              izz="0.00008508"/>
+        </inertial>
+      </link>
+      <joint name="fc_joint" type="fixed">
+        <parent link="fc_link"/>
+        <child link="fc"/>
+        <axis xyz="0 0 1"/>
+        <origin xyz="0.0129 -0.0012 0.020" rpy="0 0 0"/>
+      </joint>
     </xacro:if>
     <!-- gimbal joint -->
@@ -27,10 +67,7 @@
         <origin xyz="0.170 0 0" rpy="0 0 0" />
       </xacro:if>
-      <xacro:if value="${self == 2}">
+      <xacro:unless value="${self == 1}">
         <origin xyz="0.2035 0 0" rpy="0 0 0" />
-      </xacro:if>
-      <xacro:if value="${self == 3}">
-        <origin xyz="0.2035 0 0" rpy="0 0 0" />
-      </xacro:if>
+      </xacro:unless>
     </joint>
     <!-- link joint -->
@@ -45,19 +82,12 @@
           <origin xyz="0.494 0 0" rpy="0 0 0" />
         </xacro:if>
-        <xacro:if value="${self == 2}">
+        <xacro:unless value="${self == 1}">
           <origin xyz="0.5275 0 0" rpy="0 0 0" />
-        </xacro:if>
+        </xacro:unless>
       </joint>
     </xacro:unless>
     <!-- rotor parent (virtual) -->
     <link name="rotor_parent${self}">
-      <inertial>
-        <origin xyz="0 0 0" rpy="0 0 0"/>
-        <mass value="0.00001"/>
-        <inertia
-            ixx="0.000001" ixy="0.0" ixz="0.0"
-            iyy="0.000001" iyz="0.0"
-            izz="0.000002"/>
-      </inertial>
+      <xacro:virtual_inertial/>
     </link>
     <joint name="rotor_parent_link_joint${self}" type="fixed">
@@ -77,12 +107,5 @@
     <!-- thrust link -->
     <link name="thrust${self}">
-      <inertial>
-        <origin xyz="0 0 0" rpy="0 0 0"/>
-        <mass value="0.00001"/>
-        <inertia
-            ixx="0.000001" ixy="0.0" ixz="0.0"
-            iyy="0.000001" iyz="0.0"
-            izz="0.000002"/>
-      </inertial>
+      <xacro:virtual_inertial/>
     </link>
     <xacro:damping_factor link="thrust${self}" />
@@ -103,10 +126,7 @@
           <origin xyz="0.3735 -0.038 0" rpy="${pi / 2} 0 ${-pi / 2}"/>
         </xacro:if>
-        <xacro:if value="${self == 2}">
+        <xacro:unless value="${self == 1}">
           <origin xyz="0.407 -0.038 0" rpy="${pi / 2} 0 ${-pi / 2}"/>
-        </xacro:if>
-        <xacro:if value="${self == 3}">
-          <origin xyz="0.407 -0.038 0" rpy="${pi / 2} 0 ${-pi / 2}"/>
-        </xacro:if>
+        </xacro:unless>
       </joint>
     </xacro:if>

File: robots/delta/urdf/common.xacro (robot description, xacro)
@@ -25,5 +25,5 @@
   <!-- macro of inertial of virtual link -->
   <xacro:macro name="virtual_inertial" params="x:=0 y:=0 z:=0">
-    <inerial>
+    <inertial>
       <origin xyz="${x} ${y} ${z}"/>
       <mass value="0.00001"/>
@@ -32,5 +32,5 @@
           iyy="0.000001" iyz="0.0"
           izz="0.000002"/>
-    </inerial>
+    </inertial>
   </xacro:macro>
   <xacro:macro name="damping_factor" params="link">
