Commit message: [mini_quadrotor] tm

File: robots/mini_quadrotor/urdf/robot.urdf.xacro (robot description, xacro)
@@ -129,5 +129,5 @@
   <!-- livox mid360 -->
   <xacro:extra_module name = "lidar_imu" parent = "main_body" visible = "0" > <!-- should be IMU frame -->
-    <origin xyz="${0.011} ${0.02329} ${0.0425 + 0.047 - 0.04412}" rpy="0 0 0"/> <!-- TODO: the true pos -->
+    <origin xyz="${0.011} ${0.02329} ${0.0425 + 0.047 - 0.04412}" rpy="${pi / 2} 0 0"/> <!-- TODO: the true pos -->
     <inertial>
       <mass value = "00" />
